Commit message: compiles and starts on harmonic; plugin errors

File: urdf/4w_mecanum_waffle/base_link.urdf.xacro (robot description, xacro)
@@ -1,10 +1,10 @@
 <?xml version="1.0"?>
 <robot xmlns:xacro="http://ros.org/wiki/xacro" xmlns:ignition="http://gazebosim.com/schema">
-  <xacro:include filename="$(find ros2_omni_robot_sim)/urdf/4w_mecanum_waffle/simple_wheel.urdf.xacro"/>
-  <xacro:include filename="$(find ros2_omni_robot_sim)/urdf/4w_mecanum_waffle/mecanum_wheel.urdf.xacro"/>
-  <xacro:include filename="$(find ros2_omni_robot_sim)/urdf/4w_mecanum_waffle/camera.urdf.xacro"/>
-  <xacro:include filename="$(find ros2_omni_robot_sim)/urdf/4w_mecanum_waffle/lidar.urdf.xacro"/>
-  <xacro:include filename="$(find ros2_omni_robot_sim)/urdf/4w_mecanum_waffle/ray.urdf.xacro"/>
-  <xacro:include filename="$(find ros2_omni_robot_sim)/urdf/4w_mecanum_waffle/imu.urdf.xacro"/>
+  <xacro:include filename="$(find simbot_gz)/urdf/4w_mecanum_waffle/simple_wheel.urdf.xacro"/>
+  <xacro:include filename="$(find simbot_gz)/urdf/4w_mecanum_waffle/mecanum_wheel.urdf.xacro"/>
+  <xacro:include filename="$(find simbot_gz)/urdf/4w_mecanum_waffle/camera.urdf.xacro"/>
+  <xacro:include filename="$(find simbot_gz)/urdf/4w_mecanum_waffle/lidar.urdf.xacro"/>
+  <xacro:include filename="$(find simbot_gz)/urdf/4w_mecanum_waffle/ray.urdf.xacro"/>
+  <xacro:include filename="$(find simbot_gz)/urdf/4w_mecanum_waffle/imu.urdf.xacro"/>
   <xacro:property name="base_visual_offset" value="-0.064 0 0.047"/>
   <xacro:property name="base_collision_offset" value="-0.064 0 0.097"/>
@@ -20,5 +20,5 @@
       <origin xyz="${base_visual_offset}" rpy="0 0 0"/>
         <geometry>
-          <mesh filename="package://ros2_omni_robot_sim/meshes/waffle_base.dae" scale="0.001 0.001 0.001"/>
+          <mesh filename="package://simbot_gz/meshes/waffle_base.dae" scale="0.001 0.001 0.001"/>
         </geometry>
         <material name="red">

File: urdf/4w_mecanum_waffle/camera.urdf.xacro (robot description, xacro)
@@ -7,5 +7,5 @@
         <origin rpy="0 0 3.1416"/>
           <geometry>
-            <mesh filename="package://ros2_omni_robot_sim/meshes/camera.stl" />
+            <mesh filename="package://simbot_gz/meshes/camera.stl" />
           </geometry>
           <material name="black">
@@ -68,5 +68,5 @@
           <origin rpy="0 0 3.1416"/>
           <geometry>
-            <mesh filename="package://ros2_omni_robot_sim/meshes/camera.stl" />
+            <mesh filename="package://simbot_gz/meshes/camera.stl" />
           </geometry>
           <material name="black">

File: urdf/4w_mecanum_waffle/gazebo_plugins.urdf.xacro (robot description, xacro)
@@ -2,12 +2,12 @@
 <robot xmlns:xacro="http://ros.org/wiki/xacro">
   <gazebo>
-    <plugin filename="libignition-gazebo-sensors-system.so"
+    <plugin filename="libgz-sim-sensors-system.so"
       name="ignition::gazebo::systems::Sensors">
       <engine>ogre2</engine>
       <render_engine>optix</render_engine>
     </plugin>
-    <plugin name="ignition::gazebo::systems::Imu" filename="libignition-gazebo-imu-system.so" />
-    <plugin filename="ign_ros2_control-system" name="ign_ros2_control::IgnitionROS2ControlPlugin">
-      <parameters>$(find ros2_omni_robot_sim)/config/controller_configs/controller_config_4w_mecanum_waffle.yaml</parameters>
+    <plugin name="gazebo::sim::systems::Imu" filename="libgz-sim-imu-system.so" />
+    <plugin filename="gz_ros2_control-system" name="gz_ros2_control::GazeboSimROS2ControlPlugin">
+      <parameters>$(find simbot_gz)/config/controller_configs/controller_config_4w_mecanum_waffle.yaml</parameters>
       <ros>
         <remapping>~/odometry:=/odom</remapping>

File: urdf/4w_mecanum_waffle/main.urdf (robot description, URDF)
Before this commit: robot simple_robot, 18 links, 17 joints
Links:
- link base_link: geometry collision box size=0.266 0.266 0.094; visual mesh filename=/root/ros2_ws/src/simbot_gz/meshes/waffle_base.dae scale=0.001 0.001 0.001
- link camera_link_back: geometry collision box size=0.05 0.05 0.03; visual mesh filename=/root/ros2_ws/src/simbot_gz/meshes/camera.stl
- link camera_link_front: geometry collision box size=0.05 0.05 0.03; visual mesh filename=/root/ros2_ws/src/simbot_gz/meshes/camera.stl
- link mecanum_wheel_link_fl: geometry collision cylinder length=0.0455 radius=0.05; visual mesh filename=/root/ros2_ws/src/simbot_gz/meshes/mecanum_a.dae scale=1.0 1.0 1.0
- link mecanum_wheel_link_fr: geometry collision cylinder length=0.0455 radius=0.05; visual mesh filename=/root/ros2_ws/src/simbot_gz/meshes/mecanum_b.dae scale=1.0 1.0 1.0
- link mecanum_wheel_link_rl: geometry collision cylinder length=0.0455 radius=0.05; visual mesh filename=/root/ros2_ws/src/simbot_gz/meshes/mecanum_b.dae scale=1.0 1.0 1.0
- link mecanum_wheel_link_rr: geometry collision cylinder length=0.0455 radius=0.05; visual mesh filename=/root/ros2_ws/src/simbot_gz/meshes/mecanum_a.dae scale=1.0 1.0 1.0

File: urdf/4w_mecanum_waffle/main.urdf.xacro (robot description, xacro)
@@ -1,7 +1,7 @@
 <?xml version="1.0"?>
 <robot name="simple_robot" xmlns:xacro="http://ros.org/wiki/xacro" xmlns:ignition="http://gazebosim.com/schema">
-  <xacro:include filename="$(find ros2_omni_robot_sim)/urdf/4w_mecanum_waffle/base_link.urdf.xacro" />
-  <xacro:include filename="$(find ros2_omni_robot_sim)/urdf/4w_mecanum_waffle/gazebo_plugins.urdf.xacro" />
-  <xacro:include filename="$(find ros2_omni_robot_sim)/urdf/4w_mecanum_waffle/ros2_control.urdf.xacro" />
+  <xacro:include filename="$(find simbot_gz)/urdf/4w_mecanum_waffle/base_link.urdf.xacro" />
+  <xacro:include filename="$(find simbot_gz)/urdf/4w_mecanum_waffle/gazebo_plugins.urdf.xacro" />
+  <xacro:include filename="$(find simbot_gz)/urdf/4w_mecanum_waffle/ros2_control.urdf.xacro" />
   <link name="base_footprint" />
   <!-- <link name="base_link" /> -->

File: urdf/4w_mecanum_waffle/mecanum_wheel.urdf.xacro (robot description, xacro)
@@ -12,24 +12,24 @@
     <xacro:property name="izz" value="0.000111"/>
     <xacro:property name="visual_rotation" value="0.0"/> <!-- might be updated-->
-     <xacro:property name="mesh" value="package://ros2_omni_robot_sim/meshes/3w_v2/omni_frame.stl"/> <!-- might be updated-->
+     <xacro:property name="mesh" value="package://simbot_gz/meshes/3w_v2/omni_frame.stl"/> <!-- might be updated-->
      <xacro:property name="fdir" value="1.0 -1.0 0.0"/> <!-- might be updated-->
     <!-- Assign meshes and friction directions based on suffix -->
     <xacro:if value="${suffix_param == 'fl'}">
-      <xacro:property name="mesh" value="package://ros2_omni_robot_sim/meshes/mecanum_a.dae"/>
+      <xacro:property name="mesh" value="package://simbot_gz/meshes/mecanum_a.dae"/>
       <xacro:property name="visual_rotation" value="0.0"/>
       <xacro:property name="fdir" value="1 -1 0"/>
     </xacro:if>
     <xacro:if value="${suffix_param == 'fr'}">
-      <xacro:property name="mesh" value="package://ros2_omni_robot_sim/meshes/mecanum_b.dae"/>
+      <xacro:property name="mesh" value="package://simbot_gz/meshes/mecanum_b.dae"/>
       <xacro:property name="visual_rotation" value="0.0"/>
       <xacro:property name="fdir" value="1 1 0"/>
     </xacro:if>
     <xacro:if value="${suffix_param == 'rl'}">
-      <xacro:property name="mesh" value="package://ros2_omni_robot_sim/meshes/mecanum_b.dae"/>
+      <xacro:property name="mesh" value="package://simbot_gz/meshes/mecanum_b.dae"/>
       <xacro:property name="visual_rotation" value="0.0"/>
       <xacro:property name="fdir" value="1 1 0"/>
     </xacro:if>
     <xacro:if value="${suffix_param == 'rr'}">
-      <xacro:property name="mesh" value="package://ros2_omni_robot_sim/meshes/mecanum_a.dae"/>
+      <xacro:property name="mesh" value="package://simbot_gz/meshes/mecanum_a.dae"/>
       <xacro:property name="visual_rotation" value="0.0"/>
       <xacro:property name="fdir" value="1 -1 0"/>

File: urdf/4w_mecanum_waffle/roller.urdf.xacro (robot description, xacro)
@@ -5,5 +5,5 @@
       <visual>
         <geometry>
-          <mesh filename="package://ros2_omni_robot_sim/meshes/4w/roller.stl" />
+          <mesh filename="package://simbot_gz/meshes/4w/roller.stl" />
         </geometry>
         <material name="black">
@@ -13,5 +13,5 @@
       <collision>
         <geometry>
-          <mesh filename="package://ros2_omni_robot_sim/meshes/4w/roller.stl" />
+          <mesh filename="package://simbot_gz/meshes/4w/roller.stl" />
         </geometry>
       </collision>

File: urdf/4w_mecanum_waffle/ros2_control.urdf.xacro (robot description, xacro)
@@ -3,5 +3,5 @@
     <ros2_control name="IgnitionSystem" type="system">
         <hardware>
-            <plugin>ign_ros2_control/IgnitionSystem</plugin>
+            <plugin>gz_ros2_control/IgnitionSystem</plugin>
         </hardware>
         <joint name="mecanum_wheel_joint_fl">
