Commit message: config examples; laser collider

File: urdf/simbot_mecanum_waffle/lidar.urdf.xacro (robot description, xacro)
@@ -11,4 +11,10 @@
         </material>
       </visual>
+      <collision>
+        <origin xyz="0 0 0" rpy="0 0 0"/>
+        <geometry>
+           <cylinder radius="0.02" length="0.02" />
+        </geometry>
+      </collision>
     </link>
     <joint name="lidar_joint_${suffix}" type="fixed">
