Commit message: urdf fixes and renaming

File: urdf/simbot_mecanum_waffle/base_link.urdf.xacro (robot description, xacro)
@@ -1,10 +1,10 @@
 <?xml version="1.0"?>
 <robot xmlns:xacro="http://ros.org/wiki/xacro" xmlns:ignition="http://gazebosim.com/schema">
-  <xacro:include filename="$(find simbot_gz)/urdf/4w_mecanum_waffle/simple_wheel.urdf.xacro"/>
-  <xacro:include filename="$(find simbot_gz)/urdf/4w_mecanum_waffle/mecanum_wheel.urdf.xacro"/>
-  <xacro:include filename="$(find simbot_gz)/urdf/4w_mecanum_waffle/camera.urdf.xacro"/>
-  <xacro:include filename="$(find simbot_gz)/urdf/4w_mecanum_waffle/lidar.urdf.xacro"/>
-  <xacro:include filename="$(find simbot_gz)/urdf/4w_mecanum_waffle/ray.urdf.xacro"/>
-  <xacro:include filename="$(find simbot_gz)/urdf/4w_mecanum_waffle/imu.urdf.xacro"/>
+  <xacro:include filename="$(find simbot_gz)/urdf/simbot_mecanum_waffle/simple_wheel.urdf.xacro"/>
+  <xacro:include filename="$(find simbot_gz)/urdf/simbot_mecanum_waffle/mecanum_wheel.urdf.xacro"/>
+  <xacro:include filename="$(find simbot_gz)/urdf/simbot_mecanum_waffle/camera.urdf.xacro"/>
+  <xacro:include filename="$(find simbot_gz)/urdf/simbot_mecanum_waffle/lidar.urdf.xacro"/>
+  <xacro:include filename="$(find simbot_gz)/urdf/simbot_mecanum_waffle/ray.urdf.xacro"/>
+  <xacro:include filename="$(find simbot_gz)/urdf/simbot_mecanum_waffle/imu.urdf.xacro"/>
   <xacro:property name="base_visual_offset" value="-0.064 0 0.047"/>
   <xacro:property name="base_collision_offset" value="-0.064 0 0.097"/>
@@ -23,6 +23,6 @@
         </geometry>
         <material name="red">
- 		<color rgba="1 0 0 1" />
-	</material>
+ 		      <color rgba="1.0 0 0 1.0" />
+	      </material>
       </visual>
       <collision>
@@ -45,5 +45,5 @@
       <origin xyz="${xyz}" rpy="${rpy}" />
     </joint>
-    <!-- Childs -->
+    <!-- Wheels -->
     <!-- Front Left -->
     <xacro:mecanum_wheel parent="base_link" suffix="fl"
@@ -62,9 +62,7 @@
                         xyz="${rear_wheel_x_offset} ${right_wheel_y_offset} ${wheel_z_offset}"
                         rpy="0 0 0"/>
+    <!-- Cameras -->
     <xacro:camera2 parent="base_link" suffix="front" xyz="0.07 -0.0000 0.1030" rpy="0 0 0" visualize_model="true"/>
-    <xacro:camera2 parent="base_link" suffix="back"
-               xyz="-0.195 0.0000 0.1030"
-               rpy="0 0 3.14159"
-                visualize_model="true"/>
+    <xacro:camera2 parent="base_link" suffix="back" xyz="-0.195 0.0000 0.1030" rpy="0 0 3.14159" visualize_model="true"/>
     <!-- Top-Down Camera as moving camera -->
     <xacro:moving_camera2 parent="base_link" suffix="top"
@@ -75,8 +73,8 @@
     <xacro:lidar parent="base_link" suffix="1" xyz="0.0000 0.0000 .1510" rpy="0 0 0"/>
     <xacro:imu parent="base_link" suffix="1" xyz="0 0 0" rpy="0 0 0"/>
-    <xacro:range_sensor parent="base_link" suffix="fr" xyz="0.065 -0.10 0.08" rpy="0.0 0.0 0.0"/>
-    <xacro:range_sensor parent="base_link" suffix="fl" xyz="0.065 0.10 0.08" rpy="0.0 0.0 0.0"/>
-    <xacro:range_sensor parent="base_link" suffix="rr" xyz="-0.19 -0.10 0.08" rpy="0.0 0.0 3.1416"/>
-    <xacro:range_sensor parent="base_link" suffix="rl" xyz="-0.19 0.10 0.08" rpy="0.0 0.0 3.1416"/>
+    <xacro:range_sensor parent="base_link" suffix="fr" xyz="0.065 -0.10 0.08" rpy="0.0 0.0 -0.187"/>
+    <xacro:range_sensor parent="base_link" suffix="fl" xyz="0.065 0.10 0.08" rpy="0.0 0.0 0.187"/>
+    <xacro:range_sensor parent="base_link" suffix="rr" xyz="-0.19 -0.10 0.08" rpy="0.0 0.0 ${3.1416+0.187}"/>
+    <xacro:range_sensor parent="base_link" suffix="rl" xyz="-0.19 0.10 0.08" rpy="0.0 0.0 ${3.1416-0.187}"/>
   </xacro:macro>
 </robot>

File: urdf/simbot_mecanum_waffle/camera.urdf.xacro (robot description, xacro)
@@ -5,5 +5,5 @@
       <xacro:if value="${visualize_model}">
         <visual>
-        <origin rpy="0 0 3.1416"/>
+          <origin rpy="0 ${pi/2} ${pi}"/>
           <geometry>
             <mesh filename="package://simbot_gz/meshes/camera.stl" />
@@ -14,8 +14,8 @@
         </visual>
         <collision>
-        <origin rpy="0 0 0"/>
+          <origin xyz="0 0 0.01" rpy="0 0 0"/>
           <geometry>
-          <box size="0.05 0.05 0.03"/>
-    </geometry>
+            <box size="0.028 0.09 0.03"/>
+          </geometry>
         </collision>
     </xacro:if>
@@ -29,5 +29,5 @@
       <parent link="camera_link_${suffix}" />
       <child link="camera_optical_frame_${suffix}" />
-      <origin xyz="0 0 0" rpy="1.5708 0 1.5708"/>
+      <origin xyz="0.015 0 0.015" rpy="1.5708 0 1.5708"/>
     </joint>
     <joint name="camera_joint_${suffix}" type="fixed">

File: urdf/simbot_mecanum_waffle/gazebo_plugins.urdf.xacro (robot description, xacro)
@@ -3,5 +3,5 @@
   <gazebo>
     <plugin filename="libgz-sim-sensors-system.so"
-      name="ignition::gazebo::systems::Sensors">
+      name="gz::sim::systems::Sensors">
       <engine>ogre2</engine>
       <render_engine>optix</render_engine>
@@ -9,5 +9,5 @@
     <plugin name="gz::sim::systems::Imu" filename="gz-sim-imu-system" />
     <plugin filename="gz_ros2_control-system" name="gz_ros2_control::GazeboSimROS2ControlPlugin">
-      <parameters>$(find simbot_gz)/config/controller_configs/controller_config_4w_mecanum_waffle.yaml</parameters>
+      <parameters>$(find simbot_gz)/config/controller_configs/controller_config_simbot_mecanum_waffle.yaml</parameters>
       <ros>
         <remapping>~/odometry:=/odom</remapping>

File: urdf/simbot_mecanum_waffle/main.urdf.xacro (robot description, xacro)
@@ -1,7 +1,7 @@
 <?xml version="1.0"?>
 <robot name="simple_robot" xmlns:xacro="http://ros.org/wiki/xacro" xmlns:ignition="http://gazebosim.com/schema">
-  <xacro:include filename="$(find simbot_gz)/urdf/4w_mecanum_waffle/base_link.urdf.xacro" />
-  <xacro:include filename="$(find simbot_gz)/urdf/4w_mecanum_waffle/gazebo_plugins.urdf.xacro" />
-  <xacro:include filename="$(find simbot_gz)/urdf/4w_mecanum_waffle/ros2_control.urdf.xacro" />
+  <xacro:include filename="$(find simbot_gz)/urdf/simbot_mecanum_waffle/base_link.urdf.xacro" />
+  <xacro:include filename="$(find simbot_gz)/urdf/simbot_mecanum_waffle/gazebo_plugins.urdf.xacro" />
+  <xacro:include filename="$(find simbot_gz)/urdf/simbot_mecanum_waffle/ros2_control.urdf.xacro" />
   <link name="base_footprint" />
   <!-- <link name="base_link" /> -->

Commit message: cleanum; driving mecanum async

File: urdf/simbot_mecanum_waffle/base_link.urdf.xacro (robot description, xacro)
@@ -1,4 +1,4 @@
 <?xml version="1.0"?>
-<robot xmlns:xacro="http://ros.org/wiki/xacro" xmlns:ignition="http://gazebosim.com/schema">
+<robot xmlns:xacro="http://ros.org/wiki/xacro" xmlns:gz="http://gazebosim.com/schema">
   <xacro:include filename="$(find simbot_gz)/urdf/simbot_mecanum_waffle/simple_wheel.urdf.xacro"/>
   <xacro:include filename="$(find simbot_gz)/urdf/simbot_mecanum_waffle/mecanum_wheel.urdf.xacro"/>
@@ -7,5 +7,5 @@
   <xacro:include filename="$(find simbot_gz)/urdf/simbot_mecanum_waffle/ray.urdf.xacro"/>
   <xacro:include filename="$(find simbot_gz)/urdf/simbot_mecanum_waffle/imu.urdf.xacro"/>
-  <xacro:property name="base_visual_offset" value="-0.064 0 0.047"/>
+  <xacro:property name="base_visual_offset" value="-0.064 0 0.097"/>
   <xacro:property name="base_collision_offset" value="-0.064 0 0.097"/>
   <xacro:property name="base_collision_box_size" value="0.266 0.266 0.094"/>
@@ -20,15 +20,12 @@
       <origin xyz="${base_visual_offset}" rpy="0 0 0"/>
         <geometry>
-          <mesh filename="package://simbot_gz/meshes/waffle_base.dae" scale="0.001 0.001 0.001"/>
+          <mesh filename="package://simbot_gz/meshes/simbot_base.dae" scale="1 1 1"/>
         </geometry>
-        <material name="red">
- 		      <color rgba="1.0 0 0 1.0" />
-	      </material>
       </visual>
       <collision>
-      <origin xyz="${base_collision_offset}" rpy="0 0 0"/>
-      <geometry>
-        <box size="${base_collision_box_size}"/>
-      </geometry>
+        <origin xyz="${base_collision_offset}" rpy="0 0 0"/>
+        <geometry>
+          <box size="${base_collision_box_size}"/>
+        </geometry>
       </collision>
       <inertial>
@@ -67,5 +64,5 @@
     <!-- Top-Down Camera as moving camera -->
     <xacro:moving_camera2 parent="base_link" suffix="top"
-               xyz="0.0 0.0 0.0"
+               xyz="0.0 0.0 2.0"
                rpy="0 1.5708 0"
                visualize_model="false"

File: urdf/simbot_mecanum_waffle/camera.urdf.xacro (robot description, xacro)
@@ -51,5 +51,5 @@
             <width>1280</width>
             <height>720</height>
-	    <anti_aliasing>8</anti_aliasing>
+	          <anti_aliasing>0</anti_aliasing>
           </image>
           <clip>
@@ -62,5 +62,5 @@
   </xacro:macro>
   <!-- Macro for a moving camera with prismatic joint in z direction -->
-  <xacro:macro name="moving_camera2" params="suffix parent xyz rpy visualize_model:=true lower:=-1.0 upper:=1.0 effort:=10 velocity:=1.0">
+  <xacro:macro name="moving_camera2" params="suffix parent xyz rpy visualize_model:=true lower:=1.0 upper:=2.0 effort:=10 velocity:=1.0">
     <link name="camera_link_${suffix}">
       <xacro:if value="${visualize_model}">
@@ -112,5 +112,5 @@
             <width>1280</width>
             <height>720</height>
-            <anti_aliasing>8</anti_aliasing>
+            <anti_aliasing>0</anti_aliasing>
           </image>
           <clip>

File: urdf/simbot_mecanum_waffle/gazebo_plugins.urdf.xacro (robot description, xacro)
@@ -9,10 +9,5 @@
     <plugin name="gz::sim::systems::Imu" filename="gz-sim-imu-system" />
     <plugin filename="gz_ros2_control-system" name="gz_ros2_control::GazeboSimROS2ControlPlugin">
-      <parameters>$(find simbot_gz)/config/controller_configs/controller_config_simbot_mecanum_waffle.yaml</parameters>
-      <ros>
-        <remapping>~/odometry:=/odom</remapping>
-        <remapping>~/reference_unstamped:=/cmd_vel</remapping>
-	<remapping>~/tf_odometry:=/tf</remapping>
-      </ros>
+      <parameters>$(find simbot_gz)/config/controller_config_simbot.yaml</parameters>
     </plugin>
   </gazebo>

File: urdf/simbot_mecanum_waffle/main.urdf.xacro (robot description, xacro)
@@ -1,4 +1,4 @@
 <?xml version="1.0"?>
-<robot name="simple_robot" xmlns:xacro="http://ros.org/wiki/xacro" xmlns:ignition="http://gazebosim.com/schema">
+<robot name="simple_robot" xmlns:xacro="http://ros.org/wiki/xacro" xmlns:gz="http://gazebosim.com/schema">
   <xacro:include filename="$(find simbot_gz)/urdf/simbot_mecanum_waffle/base_link.urdf.xacro" />
   <xacro:include filename="$(find simbot_gz)/urdf/simbot_mecanum_waffle/gazebo_plugins.urdf.xacro" />

File: urdf/simbot_mecanum_waffle/mecanum_wheel.urdf.xacro (robot description, xacro)
@@ -1,4 +1,4 @@
 <?xml version="1.0" encoding="utf-8"?>
-<robot xmlns:xacro="http://www.ros.org/wiki/xacro" xmlns:ignition="http://gazebosim.com/schema">
+<robot xmlns:xacro="http://www.ros.org/wiki/xacro" xmlns:gz="http://gazebosim.com/schema">
   <!-- Parameterized Mecanum Wheel Macro -->
   <xacro:macro name="mecanum_wheel" params="parent suffix xyz rpy">
@@ -71,5 +71,5 @@
               <mu>1.0</mu>
               <mu2>0.0</mu2>
-	      <fdir1 ignition:expressed_in="base_footprint">${fdir}</fdir1>
+	            <fdir1 gz:expressed_in="base_footprint">${fdir}</fdir1>
             </ode>
           </friction>

File: urdf/simbot_mecanum_waffle/ros2_control.urdf.xacro (robot description, xacro)
@@ -1,7 +1,7 @@
 <?xml version="1.0"?>
 <robot xmlns:xacro="http://www.ros.org/wiki/xacro">
-    <ros2_control name="IgnitionSystem" type="system">
+    <ros2_control name="GazeboSimSystem" type="system">
         <hardware>
-            <plugin>gz_ros2_control/IgnitionSystem</plugin>
+            <plugin>gz_ros2_control/GazeboSimSystem</plugin>
         </hardware>
         <joint name="mecanum_wheel_joint_fl">

Commit message: shiny new body and cameras; cleanup; cameraInfo frustums fixed

File: urdf/simbot_mecanum_waffle/base_link.urdf.xacro (robot description, xacro)
@@ -65,5 +65,5 @@
     <xacro:moving_camera2 parent="base_link" suffix="top"
                xyz="0.0 0.0 2.0"
-               rpy="0 1.5708 0"
+               rpy="${pi} 0 -${pi/2}"
                visualize_model="false"
                lower="-1000" upper="1000" effort="100" velocity="100000.0"/>

File: urdf/simbot_mecanum_waffle/camera.urdf.xacro (robot description, xacro)
@@ -5,11 +5,8 @@
       <xacro:if value="${visualize_model}">
         <visual>
-          <origin rpy="0 ${pi/2} ${pi}"/>
+          <origin rpy="0 0 ${pi}"/>
           <geometry>
-            <mesh filename="package://simbot_gz/meshes/camera.stl" />
+            <mesh filename="package://simbot_gz/meshes/camera.dae" />
           </geometry>
-          <material name="black">
-            <color rgba="0 0 0 1" />
-          </material>
         </visual>
         <collision>
@@ -29,5 +26,5 @@
       <parent link="camera_link_${suffix}" />
       <child link="camera_optical_frame_${suffix}" />
-      <origin xyz="0.015 0 0.015" rpy="1.5708 0 1.5708"/>
+      <origin xyz="0.015 0 0.015" rpy="-${pi/2.0} 0 -${pi/2.0}"/>
     </joint>
     <joint name="camera_joint_${suffix}" type="fixed">
@@ -64,21 +61,4 @@
   <xacro:macro name="moving_camera2" params="suffix parent xyz rpy visualize_model:=true lower:=1.0 upper:=2.0 effort:=10 velocity:=1.0">
     <link name="camera_link_${suffix}">
-      <xacro:if value="${visualize_model}">
-        <visual>
-          <origin rpy="0 0 3.1416"/>
-          <geometry>
-            <mesh filename="package://simbot_gz/meshes/camera.stl" />
-          </geometry>
-          <material name="black">
-            <color rgba="0 0 0 1" />
-          </material>
-        </visual>
-        <collision>
-          <origin rpy="0 0 0"/>
-          <geometry>
-            <box size="0.05 0.05 0.03"/>
-          </geometry>
-        </collision>
-      </xacro:if>
       <inertial>
         <mass value="0.1" />
@@ -101,5 +81,5 @@
       <sensor name="camera_${suffix}" type="camera">
         <gz_frame_id>camera_link_${suffix}</gz_frame_id>
-        <pose>0.05 0 0 0 0 0</pose>
+        <pose>0 0 0 0 -${pi/2} ${pi/2}</pose>
         <always_on>0</always_on>
         <update_rate>30</update_rate>

Commit message: cleanup; football, floor, skybox

File: urdf/simbot_mecanum_waffle/base_link.urdf.xacro (robot description, xacro)
@@ -60,11 +60,10 @@
                         rpy="0 0 0"/>
     <!-- Cameras -->
-    <xacro:camera2 parent="base_link" suffix="front" xyz="0.07 -0.0000 0.1030" rpy="0 0 0" visualize_model="true"/>
-    <xacro:camera2 parent="base_link" suffix="back" xyz="-0.195 0.0000 0.1030" rpy="0 0 3.14159" visualize_model="true"/>
+    <xacro:robot_camera parent="base_link" suffix="front" xyz="0.07 -0.0000 0.1030" rpy="0 0 0"/>
+    <xacro:robot_camera parent="base_link" suffix="back" xyz="-0.195 0.0000 0.1030" rpy="0 0 3.14159"/> <!-- pixel_format="L8" -->
     <!-- Top-Down Camera as moving camera -->
-    <xacro:moving_camera2 parent="base_link" suffix="top"
+    <xacro:top_down_camera parent="base_link" suffix="top"
                xyz="0.0 0.0 2.0"
                rpy="${pi} 0 -${pi/2}"
-               visualize_model="false"
                lower="-1000" upper="1000" effort="100" velocity="100000.0"/>
     <xacro:lidar parent="base_link" suffix="1" xyz="0.0000 0.0000 .1510" rpy="0 0 0"/>

File: urdf/simbot_mecanum_waffle/camera.urdf.xacro (robot description, xacro)
@@ -1,24 +1,19 @@
 <?xml version="1.0"?>
 <robot xmlns:xacro="http://ros.org/wiki/xacro">
-  <xacro:macro name="camera2" params="suffix parent xyz rpy visualize_model:=true">
+  <!-- Front / back camera -->
+  <xacro:macro name="robot_camera" params="suffix parent xyz rpy pixel_format:=RGB_INT8">
     <link name="camera_link_${suffix}">
-      <xacro:if value="${visualize_model}">
-        <visual>
-          <origin rpy="0 0 ${pi}"/>
-          <geometry>
-            <mesh filename="package://simbot_gz/meshes/camera.dae" />
-          </geometry>
-        </visual>
-        <collision>
-          <origin xyz="0 0 0.01" rpy="0 0 0"/>
-          <geometry>
-            <box size="0.028 0.09 0.03"/>
-          </geometry>
-        </collision>
-    </xacro:if>
-      <inertial>
-        <mass value="0.5" />
-        <inertia ixx="0.005" ixy="0" ixz="0" iyy="0.005" iyz="0" izz="0.005" />
-      </inertial>
+      <visual>
+        <origin rpy="0 0 ${pi}"/>
+        <geometry>
+          <mesh filename="package://simbot_gz/meshes/camera.dae" />
+        </geometry>
+      </visual>
+      <collision>
+        <origin xyz="0 0 0.01" rpy="0 0 0"/>
+        <geometry>
+          <box size="0.028 0.09 0.03"/>
+        </geometry>
+      </collision>
     </link>
     <link name="camera_optical_frame_${suffix}" />
@@ -26,5 +21,5 @@
       <parent link="camera_link_${suffix}" />
       <child link="camera_optical_frame_${suffix}" />
-      <origin xyz="0.015 0 0.015" rpy="-${pi/2.0} 0 -${pi/2.0}"/>
+      <origin xyz="0.0 0 0.02" rpy="-${pi/2.0} 0 -${pi/2.0}"/>
     </joint>
     <joint name="camera_joint_${suffix}" type="fixed">
@@ -37,6 +32,6 @@
       <sensor name="camera_${suffix}" type="camera">
         <gz_frame_id>camera_optical_frame_${suffix}</gz_frame_id>
-        <pose>0.05 0 0 0 0 0</pose>
-        <always_on>0</always_on>
+        <pose>0 0 0.02 0 0 0</pose>
+        <always_on>false</always_on>
         <update_rate>30</update_rate>
         <visualize>false</visualize>
@@ -48,9 +43,10 @@
             <width>1280</width>
             <height>720</height>
-	          <anti_aliasing>0</anti_aliasing>
+            <format>${pixel_format}</format>
+	          <anti_aliasing>2</anti_aliasing>
           </image>
           <clip>
-            <near>0.1</near>
-            <far>10</far>
+            <near>0.01</near>
+            <far>100</far>
           </clip>
         </camera>
@@ -58,29 +54,18 @@
     </gazebo>
   </xacro:macro>
-  <!-- Macro for a moving camera with prismatic joint in z direction -->
-  <xacro:macro name="moving_camera2" params="suffix parent xyz rpy visualize_model:=true lower:=1.0 upper:=2.0 effort:=10 velocity:=1.0">
+  <!-- top down camera that moves in z direction -->
+  <xacro:macro name="top_down_camera" params="suffix parent xyz rpy pixel_format:=RGB_INT8 lower:=1.0 upper:=2.0 effort:=10 velocity:=1.0">
     <link name="camera_link_${suffix}">
-      <inertial>
-        <mass value="0.1" />
-        <inertia ixx="0.005" ixy="0" ixz="0" iyy="0.005" iyz="0" izz="0.005" />
-      </inertial>
-      <gravity>false</gravity>
     </link>
-    <joint name="camera_joint_${suffix}" type="prismatic">
+    <joint name="camera_joint_${suffix}" type="fixed">
       <parent link="${parent}" />
       <child link="camera_link_${suffix}" />
       <origin xyz="${xyz}" rpy="${rpy}" />
-      <axis xyz="-1 0 0"/>
-      <limit lower="${lower}" upper="${upper}" effort="${effort}" velocity="${velocity}"/>
-      <dynamics damping="10.0" friction="10.0"/>
     </joint>
-    <gazebo reference="camera_joint_${suffix}">
-      <provideFeedback>true</provideFeedback>
-    </gazebo>
     <gazebo reference="camera_link_${suffix}">
       <sensor name="camera_${suffix}" type="camera">
         <gz_frame_id>camera_link_${suffix}</gz_frame_id>
         <pose>0 0 0 0 -${pi/2} ${pi/2}</pose>
-        <always_on>0</always_on>
+        <always_on>false</always_on>
         <update_rate>30</update_rate>
         <visualize>false</visualize>
@@ -92,5 +77,6 @@
             <width>1280</width>
             <height>720</height>
-            <anti_aliasing>0</anti_aliasing>
+            <format>${pixel_format}</format>
+            <anti_aliasing>2</anti_aliasing>
           </image>
           <clip>

File: urdf/simbot_mecanum_waffle/gazebo_plugins.urdf.xacro (robot description, xacro)
@@ -2,11 +2,9 @@
 <robot xmlns:xacro="http://ros.org/wiki/xacro">
   <gazebo>
-    <plugin filename="libgz-sim-sensors-system.so"
-      name="gz::sim::systems::Sensors">
+    <plugin  name="gz::sim::systems::Sensors" filename="libgz-sim-sensors-system.so">
       <engine>ogre2</engine>
-      <render_engine>optix</render_engine>
     </plugin>
     <plugin name="gz::sim::systems::Imu" filename="gz-sim-imu-system" />
-    <plugin filename="gz_ros2_control-system" name="gz_ros2_control::GazeboSimROS2ControlPlugin">
+    <plugin name="gz_ros2_control::GazeboSimROS2ControlPlugin" filename="gz_ros2_control-system">
       <parameters>$(find simbot_gz)/config/controller_config_simbot.yaml</parameters>
     </plugin>

File: urdf/simbot_mecanum_waffle/ros2_control.urdf.xacro (robot description, xacro)
@@ -37,11 +37,4 @@
             <state_interface name="velocity" />
         </joint>
-        <joint name="camera_joint_top">
-            <command_interface name="position">
-                <param name="min">-1000.0</param>      <!-- 4m back from 5.55 -->
-                <param name="max">1000.0</param>      <!-- 4m forward from 5.55 -->
-            </command_interface>
-            <state_interface name="position"/>
-        </joint>
     </ros2_control>
 </robot>
