Commit message: wheels symmetrical from body center; odometry more reliable

File: urdf/simbot_mecanum_waffle/imu.urdf.xacro (robot description, xacro)
@@ -1,11 +1,11 @@
 <?xml version="1.0"?>
 <robot name="delirobo" xmlns:xacro="http://ros.org/wiki/xacro">
-	<xacro:macro name="imu" params="suffix parent xyz rpy">
-		<joint name="imu_joint_${suffix}" type="fixed">
+	<xacro:macro name="imu" params="parent xyz rpy">
+		<joint name="imu_joint" type="fixed">
 			<parent link="${parent}" />
-			<child link="imu_link_${suffix}" />
+			<child link="imu_link" />
 			<origin xyz="${xyz}" rpy="${rpy}" />
 		</joint>
-		<link name="imu_link_${suffix}">
+		<link name="imu_link">
 			<inertial>
 				<origin xyz="0 0 0" />
@@ -14,5 +14,5 @@
 			</inertial>
 		</link>
-		<gazebo reference="imu_link_${suffix}">
+		<gazebo reference="imu_link">
       <sensor type="imu" name="imu_sensor">
         <topic>/imu</topic>

File: urdf/simbot_mecanum_waffle/lidar.urdf.xacro (robot description, xacro)
@@ -1,6 +1,6 @@
 <?xml version="1.0"?>
 <robot xmlns:xacro="http://ros.org/wiki/xacro">
-  <xacro:macro name="lidar" params="suffix parent xyz rpy">
-    <link name="lidar_link_${suffix}">
+  <xacro:macro name="lidar" params="parent xyz rpy">
+    <link name="lidar_link">
       <visual>
         <geometry>
@@ -18,15 +18,15 @@
       </collision>
     </link>
-    <joint name="lidar_joint_${suffix}" type="fixed">
+    <joint name="lidar_joint" type="fixed">
       <parent link="${parent}" />
-      <child link="lidar_link_${suffix}" />
+      <child link="lidar_link" />
       <origin xyz="${xyz}" rpy="${rpy}" />
       <axis xyz="0 0 1" />
     </joint>
-     <gazebo reference="lidar_link_${suffix}">
+     <gazebo reference="lidar_link">
       <sensor name='gpu_lidar' type='gpu_lidar'>
         <topic>/scan</topic>
         <update_rate>30</update_rate>
-        <gz_frame_id>lidar_link_${suffix}</gz_frame_id>
+        <gz_frame_id>lidar_link</gz_frame_id>
         <ray>
           <scan>

File: urdf/simbot_mecanum_waffle/simbot_body.urdf.xacro (robot description, xacro)
@@ -8,12 +8,12 @@
   <xacro:include filename="$(find simbot_gz)/urdf/simbot_mecanum_waffle/range_sensor.urdf.xacro"/>
   <xacro:include filename="$(find simbot_gz)/urdf/simbot_mecanum_waffle/imu.urdf.xacro"/>
-  <xacro:property name="base_visual_offset" value="-0.064 0 0.097"/>
-  <xacro:property name="base_collision_offset" value="-0.064 0 0.097"/>
+  <xacro:property name="base_visual_offset" value="0 0 0.097"/>
+  <xacro:property name="base_collision_offset" value="0 0 0.097"/>
   <xacro:property name="base_collision_box_size" value="0.266 0.266 0.094"/>
   <xacro:property name="wheel_z_offset" value="0.047"/>
-  <xacro:property name="front_wheel_x_offset" value="0.015"/>
-  <xacro:property name="rear_wheel_x_offset" value="-0.15"/>
+  <xacro:property name="front_wheel_x_offset" value="0.0825"/>
+  <xacro:property name="rear_wheel_x_offset" value="-0.0825"/>
   <xacro:property name="left_wheel_y_offset" value="0.157"/>
-  <xacro:property name="right_wheel_y_offset" value="${-left_wheel_y_offset}"/>
+  <xacro:property name="right_wheel_y_offset" value="-0.157"/>
   <xacro:arg name="camera_top_z" default="2.0"/>
   <xacro:arg name="cameras_pixel_format" default="RGB_INT8"/>
@@ -57,6 +57,6 @@
       <origin xyz="${xyz}" rpy="${rpy}" />
     </joint>
-    <xacro:bumper suffix="front" xyz=".1 0 0.07" rpy="0 0 0" parent="base_link"/>
-    <xacro:bumper suffix="rear" xyz="-.225 0 0.07" rpy="0 0 ${pi}" parent="base_link"/>
+    <xacro:bumper suffix="front" xyz=".164 0 0.07" rpy="0 0 0" parent="base_link"/>
+    <xacro:bumper suffix="rear" xyz="-.164 0 0.07" rpy="0 0 ${pi}" parent="base_link"/>
     <!-- Wheels -->
     <!-- Front Left -->
@@ -85,5 +85,5 @@
       encoder_thread_count="$(arg encoder_thread_count)"
       encoder_input_pixel_format="$(arg encoder_input_pixel_format)"
-      xyz="0.07 0.0 0.1030" rpy="0 0 0"
+      xyz="0.134 0.0 0.1030" rpy="0 0 0"
       anti_aliasing="$(arg cameras_anti_aliasing)"
       bounding_boxes="true"
@@ -103,5 +103,5 @@
       encoder_thread_count="$(arg encoder_thread_count)"
       encoder_input_pixel_format="$(arg encoder_input_pixel_format)"
-      xyz="-0.195 0.0000 0.1030" rpy="0 0 3.14159"
+      xyz="-0.134 0.0000 0.1030" rpy="0 0 3.14159"
       anti_aliasing="$(arg cameras_anti_aliasing)"
       bounding_boxes="true"
@@ -121,10 +121,10 @@
       fps="$(arg cameras_fps)"
     />
-    <xacro:lidar parent="base_link" suffix="1" xyz="0.0000 0.0000 .1510" rpy="0 0 0"/>
-    <xacro:imu parent="base_link" suffix="1" xyz="-.1 0.1 .1" rpy="-${pi} ${pi} -${pi/2}"/>
-    <xacro:range_sensor parent="base_link" suffix="fr" xyz="0.065 -0.10 0.1" rpy="0.0 0.0 -0.187"/>
-    <xacro:range_sensor parent="base_link" suffix="fl" xyz="0.065 0.10 0.1" rpy="0.0 0.0 0.187"/>
-    <xacro:range_sensor parent="base_link" suffix="rr" xyz="-0.19 -0.10 0.1" rpy="0.0 0.0 ${3.1416+0.187}"/>
-    <xacro:range_sensor parent="base_link" suffix="rl" xyz="-0.19 0.10 0.1" rpy="0.0 0.0 ${3.1416-0.187}"/>
+    <xacro:lidar parent="base_link" xyz="0.064 0.0000 .1510" rpy="0 0 0"/>
+    <xacro:imu parent="base_link" xyz="-.05 0.1 .1" rpy="-${pi} ${pi} -${pi/2}"/>
+    <xacro:range_sensor parent="base_link" suffix="fr" xyz="0.129 -0.10 0.1" rpy="0.0 0.0 -0.187"/>
+    <xacro:range_sensor parent="base_link" suffix="fl" xyz="0.129 0.10 0.1" rpy="0.0 0.0 0.187"/>
+    <xacro:range_sensor parent="base_link" suffix="rr" xyz="-0.129 -0.10 0.1" rpy="0.0 0.0 ${3.1416+0.187}"/>
+    <xacro:range_sensor parent="base_link" suffix="rl" xyz="-0.129 0.10 0.1" rpy="0.0 0.0 ${3.1416-0.187}"/>
   </xacro:macro>
 </robot>
