Commit message: gazebo from source w forked gz-sensors

File: urdf/simbot_mecanum_waffle/cameras.urdf.xacro (robot description, xacro)
@@ -1,6 +1,6 @@
 <?xml version="1.0"?>
-<robot xmlns:xacro="http://ros.org/wiki/xacro">
+<robot xmlns:xacro="http://ros.org/wiki/xacro" xmlns:gz="http://gazebosim.com/schema">
   <!-- Front / back camera -->
-  <xacro:macro name="robot_camera" params="suffix parent xyz rpy pixel_format:=RGB_INT8">
+  <xacro:macro name="robot_camera" params="suffix parent xyz rpy fov:=1.2 pixel_format:=R8G8B8">
     <link name="camera_link_${suffix}">
       <visual>
@@ -39,10 +39,10 @@
         <camera>
           <camera_info_topic>rgb_${suffix}/camera_info</camera_info_topic>
-          <horizontal_fov>1.2</horizontal_fov>
+          <horizontal_fov>${fov}</horizontal_fov>
           <image>
             <width>1280</width>
             <height>720</height>
             <format>${pixel_format}</format>
-	          <anti_aliasing>2</anti_aliasing>
+            <anti_aliasing>2</anti_aliasing>
           </image>
           <clip>
@@ -54,8 +54,23 @@
     </gazebo>
   </xacro:macro>
+<!-- <gz:odometer_example>
+  <noise type="gaussian">
+    <mean>0.00001</mean>
+    <stddev>0.00001</stddev>
+  </noise>
+</gz:odometer_example> -->
+<!--
+<sensor name="camera_${suffix}" type="custom" gz:type="camera_encoder">
+  <gz_frame_id>camera_optical_frame_${suffix}</gz_frame_id>
+  <pose>0 0 0.02 0 0 0</pose>
+  <always_on>false</always_on>
+  <update_rate>30</update_rate>
+  <visualize>false</visualize>
+  <topic>rgb_${suffix}</topic>
+</sensor>
+-->
   <!-- top down camera that moves in z direction -->
-  <xacro:macro name="top_down_camera" params="suffix parent xyz rpy pixel_format:=RGB_INT8 lower:=1.0 upper:=2.0 effort:=10 velocity:=1.0">
-    <link name="camera_link_${suffix}">
-    </link>
+  <xacro:macro name="top_down_camera" params="suffix parent xyz rpy pixel_format:=R8G8B8 lower:=1.0 upper:=2.0 effort:=10 velocity:=1.0">
+    <link name="camera_link_${suffix}"/>
     <joint name="camera_joint_${suffix}" type="fixed">
       <parent link="${parent}" />
@@ -85,4 +100,9 @@
           </clip>
         </camera>
+        <!-- <plugin
+          filename="gz-sim-camera-video-recorder-system"
+          name="gz::sim::systems::CameraVideoRecorder">
+          <service>camera/record_video</service>
+        </plugin> -->
       </sensor>
     </gazebo>

File: urdf/simbot_mecanum_waffle/gazebo_plugins.urdf.xacro (robot description, xacro)
@@ -3,5 +3,5 @@
   <gazebo>
     <plugin  name="gz::sim::systems::Sensors" filename="libgz-sim-sensors-system.so">
-      <engine>ogre2</engine>
+      <render_engine>ogre2</render_engine>
     </plugin>
     <plugin name="gz::sim::systems::Imu" filename="gz-sim-imu-system" />

File: urdf/simbot_mecanum_waffle/main.urdf.xacro (robot description, xacro)
@@ -1,6 +1,6 @@
 <?xml version="1.0"?>
-<robot name="simple_robot" xmlns:xacro="http://ros.org/wiki/xacro" xmlns:gz="http://gazebosim.com/schema">
-  <xacro:include filename="$(find simbot_gz)/urdf/simbot_mecanum_waffle/base_link.urdf.xacro" />
+<robot name="phntm_simbot" xmlns:xacro="http://ros.org/wiki/xacro" xmlns:gz="http://gazebosim.com/schema">
   <xacro:include filename="$(find simbot_gz)/urdf/simbot_mecanum_waffle/gazebo_plugins.urdf.xacro" />
+  <xacro:include filename="$(find simbot_gz)/urdf/simbot_mecanum_waffle/simbot_body.urdf.xacro" />
   <xacro:include filename="$(find simbot_gz)/urdf/simbot_mecanum_waffle/ros2_control.urdf.xacro" />
   <link name="base_footprint" />

File: urdf/simbot_mecanum_waffle/simbot_body.urdf.xacro (robot description, xacro)
@@ -1,7 +1,7 @@
 <?xml version="1.0"?>
 <robot xmlns:xacro="http://ros.org/wiki/xacro" xmlns:gz="http://gazebosim.com/schema">
-  <xacro:include filename="$(find simbot_gz)/urdf/simbot_mecanum_waffle/simple_wheel.urdf.xacro"/>
+  <!-- <xacro:include filename="$(find simbot_gz)/urdf/simbot_mecanum_waffle/simple_wheel.urdf.xacro"/> -->
   <xacro:include filename="$(find simbot_gz)/urdf/simbot_mecanum_waffle/mecanum_wheel.urdf.xacro"/>
-  <xacro:include filename="$(find simbot_gz)/urdf/simbot_mecanum_waffle/camera.urdf.xacro"/>
+  <xacro:include filename="$(find simbot_gz)/urdf/simbot_mecanum_waffle/cameras.urdf.xacro"/>
   <xacro:include filename="$(find simbot_gz)/urdf/simbot_mecanum_waffle/lidar.urdf.xacro"/>
   <xacro:include filename="$(find simbot_gz)/urdf/simbot_mecanum_waffle/ray.urdf.xacro"/>
@@ -59,8 +59,8 @@
                         xyz="${rear_wheel_x_offset} ${right_wheel_y_offset} ${wheel_z_offset}"
                         rpy="0 0 0"/>
-    <!-- Cameras -->
-    <xacro:robot_camera parent="base_link" suffix="front" xyz="0.07 -0.0000 0.1030" rpy="0 0 0"/>
+    <!-- Robot cameras -->
+    <xacro:robot_camera parent="base_link" suffix="front" xyz="0.07 -0.0000 0.1030" rpy="0 0 0" fov="1.5"/>
     <xacro:robot_camera parent="base_link" suffix="back" xyz="-0.195 0.0000 0.1030" rpy="0 0 3.14159"/> <!-- pixel_format="L8" -->
-    <!-- Top-Down Camera as moving camera -->
+    <!-- Top-Down camera as moving camera -->
     <xacro:top_down_camera parent="base_link" suffix="top"
                xyz="0.0 0.0 2.0"

Commit message: wide camera fix

File: urdf/simbot_mecanum_waffle/cameras.urdf.xacro (robot description, xacro)
@@ -13,5 +13,5 @@
         <origin xyz="0 0 0.01" rpy="0 0 0"/>
         <geometry>
-          <box size="0.028 0.09 0.03"/>
+          <box size="0.035 0.09 0.03"/>
         </geometry>
       </collision>
@@ -47,5 +47,5 @@
           </image>
           <clip>
-            <near>0.01</near>
+            <near>0.015</near>
             <far>100</far>
           </clip>

Commit message: fixes, tweaks and cleanup; sim extras back; range sensors faster + producing 0 when > max

File: urdf/simbot_mecanum_waffle/cameras.urdf.xacro (robot description, xacro)
@@ -2,5 +2,5 @@
 <robot xmlns:xacro="http://ros.org/wiki/xacro" xmlns:gz="http://gazebosim.com/schema">
   <!-- Front / back camera -->
-  <xacro:macro name="robot_camera" params="suffix parent xyz rpy fov:=1.2 pixel_format:=R8G8B8">
+  <xacro:macro name="robot_camera" params="suffix parent xyz rpy fov:=1.2 pixel_format:=RGB_INT8">
     <link name="camera_link_${suffix}">
       <visual>
@@ -40,5 +40,4 @@
           <camera_info_topic>rgb_${suffix}/camera_info</camera_info_topic>
           <camera_h264_topic>rgb_${suffix}/h264</camera_h264_topic>
-          <lazy>true</lazy>
           <horizontal_fov>${fov}</horizontal_fov>
           <image>
@@ -46,5 +45,5 @@
             <height>720</height>
             <format>${pixel_format}</format>
-            <anti_aliasing>2</anti_aliasing>
+            <anti_aliasing>4</anti_aliasing>
           </image>
           <clip>
@@ -73,5 +72,5 @@
 -->
   <!-- top down camera that moves in z direction -->
-  <xacro:macro name="top_down_camera" params="suffix parent xyz rpy pixel_format:=R8G8B8 lower:=1.0 upper:=2.0 effort:=10 velocity:=1.0">
+  <xacro:macro name="top_down_camera" params="suffix parent xyz rpy pixel_format:=RGB_INT8 lower:=1.0 upper:=2.0 effort:=10 velocity:=1.0">
     <link name="camera_link_${suffix}"/>
     <joint name="camera_joint_${suffix}" type="fixed">
@@ -91,5 +90,4 @@
           <camera_info_topic>rgb_${suffix}/camera_info</camera_info_topic>
           <camera_h264_topic>rgb_${suffix}/h264</camera_h264_topic>
-          <lazy>true</lazy>
           <horizontal_fov>1.2</horizontal_fov>
           <image>
@@ -97,5 +95,5 @@
             <height>720</height>
             <format>${pixel_format}</format>
-            <anti_aliasing>2</anti_aliasing>
+            <anti_aliasing>4</anti_aliasing>
           </image>
           <clip>

File: urdf/simbot_mecanum_waffle/simbot_body.urdf.xacro (robot description, xacro)
@@ -5,5 +5,5 @@
   <xacro:include filename="$(find simbot_gz)/urdf/simbot_mecanum_waffle/cameras.urdf.xacro"/>
   <xacro:include filename="$(find simbot_gz)/urdf/simbot_mecanum_waffle/lidar.urdf.xacro"/>
-  <xacro:include filename="$(find simbot_gz)/urdf/simbot_mecanum_waffle/ray.urdf.xacro"/>
+  <xacro:include filename="$(find simbot_gz)/urdf/simbot_mecanum_waffle/range_sensor.urdf.xacro"/>
   <xacro:include filename="$(find simbot_gz)/urdf/simbot_mecanum_waffle/imu.urdf.xacro"/>
   <xacro:property name="base_visual_offset" value="-0.064 0 0.097"/>
@@ -61,10 +61,7 @@
     <!-- Robot cameras -->
     <xacro:robot_camera parent="base_link" suffix="front" fov="1.5" xyz="0.07 -0.0000 0.1030" rpy="0 0 0"/>
-    <xacro:robot_camera parent="base_link" suffix="back" pixel_format="RGB_INT8" xyz="-0.195 0.0000 0.1030" rpy="0 0 3.14159"/> <!-- pixel_format="L8" -->
+    <xacro:robot_camera parent="base_link" suffix="back" xyz="-0.195 0.0000 0.1030" rpy="0 0 3.14159"/> <!-- pixel_format="L8" -->
     <!-- Top-Down camera as moving camera -->
-    <xacro:top_down_camera parent="base_link" suffix="top"
-               xyz="0.0 0.0 2.0"
-               rpy="${pi} 0 -${pi/2}"
-               lower="-1000" upper="1000" effort="100" velocity="100000.0"/>
+    <xacro:top_down_camera parent="base_link" suffix="top" xyz="0.0 0.0 2.0" rpy="${pi} 0 -${pi/2}"/>
     <xacro:lidar parent="base_link" suffix="1" xyz="0.0000 0.0000 .1510" rpy="0 0 0"/>
     <xacro:imu parent="base_link" suffix="1" xyz="0 0 0" rpy="0 0 0"/>

Commit message: porametrized camera rendering settings, readme, top camera Z ediatble via argument

File: urdf/simbot_mecanum_waffle/cameras.urdf.xacro (robot description, xacro)
@@ -2,5 +2,5 @@
 <robot xmlns:xacro="http://ros.org/wiki/xacro" xmlns:gz="http://gazebosim.com/schema">
   <!-- Front / back camera -->
-  <xacro:macro name="robot_camera" params="suffix parent xyz rpy fov:=1.2 pixel_format:=RGB_INT8">
+  <xacro:macro name="robot_camera" params="suffix parent xyz rpy fov:=1.2 pixel_format:=RGB_INT8 encoder_hw_device:=cuda encoder_bit_rate:=1000000 encoder_thread_count:=2 encoder_input_pixel_format">
     <link name="camera_link_${suffix}">
       <visual>
@@ -41,4 +41,8 @@
           <camera_h264_topic>rgb_${suffix}/h264</camera_h264_topic>
           <horizontal_fov>${fov}</horizontal_fov>
+          <encoder_hw_device>${encoder_hw_device}</encoder_hw_device>
+          <encoder_bit_rate>${encoder_bit_rate}</encoder_bit_rate>
+          <encoder_input_pixel_format>${encoder_input_pixel_format}</encoder_input_pixel_format>
+          <encoder_thread_count>${encoder_thread_count}</encoder_thread_count>
           <image>
             <width>1280</width>
@@ -72,5 +76,5 @@
 -->
   <!-- top down camera that moves in z direction -->
-  <xacro:macro name="top_down_camera" params="suffix parent xyz rpy pixel_format:=RGB_INT8 lower:=1.0 upper:=2.0 effort:=10 velocity:=1.0">
+  <xacro:macro name="top_down_camera" params="suffix parent xyz rpy pixel_format:=RGB_INT8 encoder_hw_device:=cuda encoder_bit_rate:=1000000 encoder_thread_count:=2 encoder_input_pixel_format">
     <link name="camera_link_${suffix}"/>
     <joint name="camera_joint_${suffix}" type="fixed">
@@ -91,4 +95,8 @@
           <camera_h264_topic>rgb_${suffix}/h264</camera_h264_topic>
           <horizontal_fov>1.2</horizontal_fov>
+          <encoder_hw_device>${encoder_hw_device}</encoder_hw_device>
+          <encoder_bit_rate>${encoder_bit_rate}</encoder_bit_rate>
+          <encoder_input_pixel_format>${encoder_input_pixel_format}</encoder_input_pixel_format>
+          <encoder_thread_count>${encoder_thread_count}</encoder_thread_count>
           <image>
             <width>1280</width>
@@ -99,5 +107,5 @@
           <clip>
             <near>0.1</near>
-            <far>10</far>
+            <far>100</far>
           </clip>
         </camera>

File: urdf/simbot_mecanum_waffle/simbot_body.urdf.xacro (robot description, xacro)
@@ -15,4 +15,10 @@
   <xacro:property name="left_wheel_y_offset" value="0.157"/>
   <xacro:property name="right_wheel_y_offset" value="${-left_wheel_y_offset}"/>
+  <xacro:arg name="camera_top_z" default="2.0"/>
+  <xacro:arg name="cameras_pixel_format" default="RGB_INT8"/>
+  <xacro:arg name="encoder_hw_device" default="cuda"/>
+  <xacro:arg name="encoder_bit_rate" default="1000000"/>
+  <xacro:arg name="encoder_input_pixel_format" default=""/>
+  <xacro:arg name="encoder_thread_count" default="2"/>
   <xacro:macro name="base_link" params="parent xyz rpy">
     <link name="base_link">
@@ -60,8 +66,29 @@
                         rpy="0 0 0"/>
     <!-- Robot cameras -->
-    <xacro:robot_camera parent="base_link" suffix="front" fov="1.5" xyz="0.07 -0.0000 0.1030" rpy="0 0 0"/>
-    <xacro:robot_camera parent="base_link" suffix="back" xyz="-0.195 0.0000 0.1030" rpy="0 0 3.14159"/> <!-- pixel_format="L8" -->
+    <xacro:robot_camera parent="base_link" suffix="front" fov="1.5"
+      pixel_format="$(arg cameras_pixel_format)"
+      encoder_hw_device="$(arg encoder_hw_device)"
+      encoder_bit_rate="$(arg encoder_bit_rate)"
+      encoder_thread_count="$(arg encoder_thread_count)"
+      encoder_input_pixel_format="$(arg encoder_input_pixel_format)"
+      xyz="0.07 -0.0000 0.1030" rpy="0 0 0"
+    />
+    <xacro:robot_camera parent="base_link" suffix="back"
+      pixel_format="$(arg cameras_pixel_format)"
+      encoder_hw_device="$(arg encoder_hw_device)"
+      encoder_bit_rate="$(arg encoder_bit_rate)"
+      encoder_thread_count="$(arg encoder_thread_count)"
+      encoder_input_pixel_format="$(arg encoder_input_pixel_format)"
+      xyz="-0.195 0.0000 0.1030" rpy="0 0 3.14159"
+    /> <!-- pixel_format="L8" -->
     <!-- Top-Down camera as moving camera -->
-    <xacro:top_down_camera parent="base_link" suffix="top" xyz="0.0 0.0 2.0" rpy="${pi} 0 -${pi/2}"/>
+    <xacro:top_down_camera parent="base_link" suffix="top"
+      pixel_format="$(arg cameras_pixel_format)"
+      encoder_hw_device="$(arg encoder_hw_device)"
+      encoder_bit_rate="$(arg encoder_bit_rate)"
+      encoder_thread_count="$(arg encoder_thread_count)"
+      encoder_input_pixel_format="$(arg encoder_input_pixel_format)"
+      xyz="0.0 0.0 $(arg camera_top_z)" rpy="${pi} 0 -${pi/2}"
+    />
     <xacro:lidar parent="base_link" suffix="1" xyz="0.0000 0.0000 .1510" rpy="0 0 0"/>
     <xacro:imu parent="base_link" suffix="1" xyz="0 0 0" rpy="0 0 0"/>

Commit message: building from binaries + custom packages from source; cameras_resolution param; tested on jetson orin nano

File: urdf/simbot_mecanum_waffle/cameras.urdf.xacro (robot description, xacro)
@@ -2,5 +2,5 @@
 <robot xmlns:xacro="http://ros.org/wiki/xacro" xmlns:gz="http://gazebosim.com/schema">
   <!-- Front / back camera -->
-  <xacro:macro name="robot_camera" params="suffix parent xyz rpy fov:=1.2 pixel_format:=RGB_INT8 encoder_hw_device:=cuda encoder_bit_rate:=1000000 encoder_thread_count:=2 encoder_input_pixel_format">
+  <xacro:macro name="robot_camera" params="suffix parent xyz rpy fov:=1.2 width height pixel_format:=RGB_INT8 encoder_hw_device:=cuda encoder_bit_rate:=1000000 encoder_thread_count:=2 encoder_input_pixel_format">
     <link name="camera_link_${suffix}">
       <visual>
@@ -46,6 +46,6 @@
           <encoder_thread_count>${encoder_thread_count}</encoder_thread_count>
           <image>
-            <width>1280</width>
-            <height>720</height>
+            <width>${width}</width>
+            <height>${height}</height>
             <format>${pixel_format}</format>
             <anti_aliasing>4</anti_aliasing>
@@ -76,5 +76,5 @@
 -->
   <!-- top down camera that moves in z direction -->
-  <xacro:macro name="top_down_camera" params="suffix parent xyz rpy pixel_format:=RGB_INT8 encoder_hw_device:=cuda encoder_bit_rate:=1000000 encoder_thread_count:=2 encoder_input_pixel_format">
+  <xacro:macro name="top_down_camera" params="suffix parent xyz rpy width height pixel_format:=RGB_INT8 encoder_hw_device:=cuda encoder_bit_rate:=1000000 encoder_thread_count:=2 encoder_input_pixel_format">
     <link name="camera_link_${suffix}"/>
     <joint name="camera_joint_${suffix}" type="fixed">
@@ -100,6 +100,6 @@
           <encoder_thread_count>${encoder_thread_count}</encoder_thread_count>
           <image>
-            <width>1280</width>
-            <height>720</height>
+            <width>${width}</width>
+            <height>${height}</height>
             <format>${pixel_format}</format>
             <anti_aliasing>4</anti_aliasing>

File: urdf/simbot_mecanum_waffle/simbot_body.urdf.xacro (robot description, xacro)
@@ -21,4 +21,6 @@
   <xacro:arg name="encoder_input_pixel_format" default=""/>
   <xacro:arg name="encoder_thread_count" default="2"/>
+  <xacro:arg name="cameras_width" default="1280"/>
+  <xacro:arg name="cameras_height" default="720"/>
   <xacro:macro name="base_link" params="parent xyz rpy">
     <link name="base_link">
@@ -67,4 +69,6 @@
     <!-- Robot cameras -->
     <xacro:robot_camera parent="base_link" suffix="front" fov="1.5"
+      width="$(arg cameras_width)"
+      height="$(arg cameras_height)"
       pixel_format="$(arg cameras_pixel_format)"
       encoder_hw_device="$(arg encoder_hw_device)"
@@ -75,4 +79,6 @@
     />
     <xacro:robot_camera parent="base_link" suffix="back"
+      width="$(arg cameras_width)"
+      height="$(arg cameras_height)"
       pixel_format="$(arg cameras_pixel_format)"
       encoder_hw_device="$(arg encoder_hw_device)"
@@ -84,4 +90,6 @@
     <!-- Top-Down camera as moving camera -->
     <xacro:top_down_camera parent="base_link" suffix="top"
+      width="$(arg cameras_width)"
+      height="$(arg cameras_height)"
       pixel_format="$(arg cameras_pixel_format)"
       encoder_hw_device="$(arg encoder_hw_device)"

Commit message: nls win to linux; defaults for amd encoder; symlinking python scripts on colcon build --symlink-install

File: urdf/simbot_mecanum_waffle/cameras.urdf.xacro (robot description, xacro)
@@ -2,5 +2,5 @@
 <robot xmlns:xacro="http://ros.org/wiki/xacro" xmlns:gz="http://gazebosim.com/schema">
   <!-- Front / back camera -->
-  <xacro:macro name="robot_camera" params="suffix parent xyz rpy fov:=1.2 width height pixel_format:=RGB_INT8 encoder_hw_device:=cuda encoder_bit_rate:=1000000 encoder_thread_count:=2 encoder_input_pixel_format">
+  <xacro:macro name="robot_camera" params="suffix parent xyz rpy fov:=1.2 width height pixel_format encoder_hw_device encoder_bit_rate encoder_thread_count encoder_input_pixel_format anti_aliasing">
     <link name="camera_link_${suffix}">
       <visual>
@@ -36,5 +36,5 @@
         <update_rate>30</update_rate>
         <visualize>false</visualize>
-        <topic>rgb_${suffix}</topic>
+        <topic>rgb_${suffix}/raw</topic>
         <camera>
           <camera_info_topic>rgb_${suffix}/camera_info</camera_info_topic>
@@ -49,5 +49,5 @@
             <height>${height}</height>
             <format>${pixel_format}</format>
-            <anti_aliasing>4</anti_aliasing>
+            <anti_aliasing>${anti_aliasing}</anti_aliasing>
           </image>
           <clip>
@@ -60,5 +60,5 @@
   </xacro:macro>
   <!-- top down camera that moves in z direction -->
-  <xacro:macro name="top_down_camera" params="suffix parent xyz rpy width height pixel_format:=RGB_INT8 encoder_hw_device:=cuda encoder_bit_rate:=1000000 encoder_thread_count:=2 encoder_input_pixel_format">
+  <xacro:macro name="top_down_camera" params="suffix parent xyz rpy width height pixel_format encoder_hw_device encoder_bit_rate encoder_thread_count encoder_input_pixel_format anti_aliasing">
     <link name="camera_link_${suffix}"/>
     <joint name="camera_joint_${suffix}" type="fixed">
@@ -74,5 +74,5 @@
         <update_rate>30</update_rate>
         <visualize>false</visualize>
-        <topic>rgb_${suffix}</topic>
+        <topic>rgb_${suffix}/raw</topic>
         <camera>
           <camera_info_topic>rgb_${suffix}/camera_info</camera_info_topic>
@@ -87,5 +87,5 @@
             <height>${height}</height>
             <format>${pixel_format}</format>
-            <anti_aliasing>4</anti_aliasing>
+            <anti_aliasing>${anti_aliasing}</anti_aliasing>
           </image>
           <clip>

File: urdf/simbot_mecanum_waffle/simbot_body.urdf.xacro (robot description, xacro)
@@ -23,4 +23,5 @@
   <xacro:arg name="cameras_width" default="1280"/>
   <xacro:arg name="cameras_height" default="720"/>
+  <xacro:arg name="cameras_anti_aliasing" default="4"/>
   <xacro:macro name="base_link" params="parent xyz rpy">
     <link name="base_link">
@@ -77,4 +78,5 @@
       encoder_input_pixel_format="$(arg encoder_input_pixel_format)"
       xyz="0.07 -0.0000 0.1030" rpy="0 0 0"
+      anti_aliasing="$(arg cameras_anti_aliasing)"
     />
     <xacro:robot_camera parent="base_link" suffix="back"
@@ -87,4 +89,5 @@
       encoder_input_pixel_format="$(arg encoder_input_pixel_format)"
       xyz="-0.195 0.0000 0.1030" rpy="0 0 3.14159"
+      anti_aliasing="$(arg cameras_anti_aliasing)"
     /> <!-- pixel_format="L8" -->
     <!-- Top-Down camera as moving camera -->
@@ -98,4 +101,5 @@
       encoder_input_pixel_format="$(arg encoder_input_pixel_format)"
       xyz="0.0 0.0 $(arg camera_top_z)" rpy="${pi} 0 -${pi/2}"
+      anti_aliasing="$(arg cameras_anti_aliasing)"
     />
     <xacro:lidar parent="base_link" suffix="1" xyz="0.0000 0.0000 .1510" rpy="0 0 0"/>
