Commit message: readme, updated with depth a camera

File: urdf/simbot_mecanum_waffle/cameras.urdf.xacro (robot description, xacro)
@@ -2,5 +2,5 @@
 <robot xmlns:xacro="http://ros.org/wiki/xacro" xmlns:gz="http://gazebosim.com/schema">
   <!-- Front / back camera -->
-  <xacro:macro name="robot_camera" params="suffix parent xyz rpy fov:=1.2 width height pixel_format encoder_hw_device encoder_bit_rate encoder_thread_count encoder_input_pixel_format anti_aliasing">
+  <xacro:macro name="robot_camera" params="suffix parent xyz rpy fov:=1.2 width height pixel_format encoder_hw_device encoder_bit_rate encoder_thread_count encoder_input_pixel_format anti_aliasing depth:=false">
     <link name="camera_link_${suffix}">
       <visual>
@@ -17,10 +17,4 @@
       </collision>
     </link>
-    <link name="camera_optical_frame_${suffix}" />
-    <joint name="camera_optical_joint_${suffix}" type="fixed">
-      <parent link="camera_link_${suffix}" />
-      <child link="camera_optical_frame_${suffix}" />
-      <origin xyz="0.0 0 0.02" rpy="-${pi/2.0} 0 -${pi/2.0}"/>
-    </joint>
     <joint name="camera_joint_${suffix}" type="fixed">
       <parent link="${parent}" />
@@ -29,8 +23,14 @@
       <axis xyz="0 0 1"/>
     </joint>
-    <gazebo reference="camera_link_${suffix}">
+    <link name="camera_optical_frame_${suffix}" />
+    <joint name="camera_optical_joint_${suffix}" type="fixed">
+      <parent link="camera_link_${suffix}" />
+      <child link="camera_optical_frame_${suffix}" />
+      <origin xyz="0.012 0.03 0.015" rpy="-${pi/2.0} 0 -${pi/2.0}"/>
+    </joint>
+    <gazebo reference="camera_optical_frame_${suffix}">
       <sensor name="camera_${suffix}" type="camera">
         <gz_frame_id>camera_optical_frame_${suffix}</gz_frame_id>
-        <pose>0 0 0.02 0 0 0</pose>
+        <pose>0 0 0 0 -${pi/2.0} ${pi/2.0}</pose>
         <always_on>true</always_on>
         <update_rate>30</update_rate>
@@ -52,5 +52,5 @@
           </image>
           <clip>
-            <near>0.015</near>
+            <near>0.001</near> <!-- less than collider to prevent seeing through walls -->
             <far>100</far>
           </clip>
@@ -58,4 +58,35 @@
       </sensor>
     </gazebo>
+    <!-- Depth camera -->
+    <xacro:if value="${depth}">
+      <link name="depth_camera_optical_frame_${suffix}" />
+      <joint name="depth_camera_optical_joint_${suffix}" type="fixed">
+        <parent link="camera_link_${suffix}" />
+        <child link="depth_camera_optical_frame_${suffix}" />
+        <origin xyz="0.012 -0.03 0.015" rpy="-${pi/2.0} 0 -${pi/2.0}"/>
+      </joint>
+      <gazebo reference="depth_camera_optical_frame_${suffix}">
+        <sensor name="depth_camera_${suffix}" type="depth_camera">
+          <gz_frame_id>depth_camera_optical_frame_${suffix}</gz_frame_id>
+          <pose>0 0 0 -${pi/2.0} ${pi/2.0}</pose>
+          <always_on>true</always_on>
+          <update_rate>30</update_rate>
+          <visualize>false</visualize>
+          <topic>depth_${suffix}/raw</topic>
+          <camera>
+            <camera_info_topic>depth_${suffix}/camera_info</camera_info_topic>
+            <horizontal_fov>${fov}</horizontal_fov>
+            <image>
+              <width>640</width>
+              <height>480</height>
+            </image>
+            <clip>
+              <near>0.1</near> <!-- smaller produces rendering errors -->
+              <far>100</far>
+            </clip>
+          </camera>
+        </sensor>
+      </gazebo>
+    </xacro:if>
   </xacro:macro>
   <!-- top down camera that moves in z direction -->

File: urdf/simbot_mecanum_waffle/simbot_body.urdf.xacro (robot description, xacro)
@@ -18,5 +18,5 @@
   <xacro:arg name="cameras_pixel_format" default="RGB_INT8"/>
   <xacro:arg name="encoder_hw_device" default="cuda"/>
-  <xacro:arg name="encoder_bit_rate" default="1000000"/>
+  <xacro:arg name="encoder_bit_rate" default="2000000"/>
   <xacro:arg name="encoder_input_pixel_format" default=""/>
   <xacro:arg name="encoder_thread_count" default="2"/>
@@ -77,6 +77,7 @@
       encoder_thread_count="$(arg encoder_thread_count)"
       encoder_input_pixel_format="$(arg encoder_input_pixel_format)"
-      xyz="0.07 -0.0000 0.1030" rpy="0 0 0"
+      xyz="0.07 0.0 0.1030" rpy="0 0 0"
       anti_aliasing="$(arg cameras_anti_aliasing)"
+      depth="true"
     />
     <xacro:robot_camera parent="base_link" suffix="back"

Commit message: updates and tweaks; bb cameras, rendering at ~30 FPS w 3 cameras

File: urdf/simbot_mecanum_waffle/cameras.urdf.xacro (robot description, xacro)
@@ -2,5 +2,5 @@
 <robot xmlns:xacro="http://ros.org/wiki/xacro" xmlns:gz="http://gazebosim.com/schema">
   <!-- Front / back camera -->
-  <xacro:macro name="robot_camera" params="suffix parent xyz rpy fov:=1.2 width height pixel_format encoder_hw_device encoder_bit_rate encoder_thread_count encoder_input_pixel_format anti_aliasing depth:=false">
+  <xacro:macro name="robot_camera" params="suffix parent xyz rpy fov:=1.2 width height pixel_format encoder_hw_device encoder_bit_rate encoder_thread_count encoder_input_pixel_format anti_aliasing depth:=false fps:=90 bounding_boxes:=false">
     <link name="camera_link_${suffix}">
       <visual>
@@ -34,5 +34,5 @@
         <pose>0 0 0 0 -${pi/2.0} ${pi/2.0}</pose>
         <always_on>true</always_on>
-        <update_rate>30</update_rate>
+        <update_rate>${fps}</update_rate>
         <visualize>false</visualize>
         <topic>rgb_${suffix}/raw</topic>
@@ -45,4 +45,5 @@
           <encoder_input_pixel_format>${encoder_input_pixel_format}</encoder_input_pixel_format>
           <encoder_thread_count>${encoder_thread_count}</encoder_thread_count>
+          <bounding_boxes>${bounding_boxes}</bounding_boxes>
           <image>
             <width>${width}</width>
@@ -57,4 +58,29 @@
         </camera>
       </sensor>
+      <!-- BB camera -->
+      <xacro:if value="${bounding_boxes}">
+        <sensor name="bb_camera_${suffix}" type="boundingbox_camera">
+          <gz_frame_id>camera_optical_frame_${suffix}</gz_frame_id>
+          <always_on>true</always_on>
+          <pose>0 0 0 0 -${pi/2.0} ${pi/2.0}</pose>
+          <update_rate>${fps}</update_rate>
+          <visualize>true</visualize>
+          <topic>bb_${suffix}/this_must_be_here</topic>
+          <camera>
+            <topic2d>detections/${suffix}/boxes_2d</topic2d>
+            <topic3d>detections/${suffix}/boxes_3d</topic3d>
+            <box_type>2d+3d</box_type>
+            <horizontal_fov>${fov}</horizontal_fov>
+            <image>
+              <width>${width/10}</width>
+              <height>${height/10}</height>
+            </image>
+            <clip>
+              <near>0.001</near>
+              <far>10</far>
+            </clip>
+          </camera>
+        </sensor>
+      </xacro:if>
     </gazebo>
     <!-- Depth camera -->
@@ -69,7 +95,7 @@
         <sensor name="depth_camera_${suffix}" type="depth_camera">
           <gz_frame_id>depth_camera_optical_frame_${suffix}</gz_frame_id>
-          <pose>0 0 0 -${pi/2.0} ${pi/2.0}</pose>
+          <pose>0 0 0 0 -${pi/2.0} ${pi/2.0}</pose>
           <always_on>true</always_on>
-          <update_rate>30</update_rate>
+          <update_rate>${fps}</update_rate>
           <visualize>false</visualize>
           <topic>depth_${suffix}/raw</topic>
@@ -91,5 +117,5 @@
   </xacro:macro>
   <!-- top down camera that moves in z direction -->
-  <xacro:macro name="top_down_camera" params="suffix parent xyz rpy width height pixel_format encoder_hw_device encoder_bit_rate encoder_thread_count encoder_input_pixel_format anti_aliasing">
+  <xacro:macro name="top_down_camera" params="suffix parent xyz rpy width height pixel_format encoder_hw_device encoder_bit_rate encoder_thread_count encoder_input_pixel_format anti_aliasing fps:=90">
     <link name="camera_link_${suffix}"/>
     <joint name="camera_joint_${suffix}" type="fixed">
@@ -103,5 +129,5 @@
         <pose>0 0 0 0 -${pi/2} ${pi/2}</pose>
         <always_on>true</always_on>
-        <update_rate>30</update_rate>
+        <update_rate>${fps}</update_rate>
         <visualize>false</visualize>
         <topic>rgb_${suffix}/raw</topic>

File: urdf/simbot_mecanum_waffle/simbot_body.urdf.xacro (robot description, xacro)
@@ -80,4 +80,5 @@
       anti_aliasing="$(arg cameras_anti_aliasing)"
       depth="true"
+      bounding_boxes="true"
     />
     <xacro:robot_camera parent="base_link" suffix="back"
@@ -91,4 +92,5 @@
       xyz="-0.195 0.0000 0.1030" rpy="0 0 3.14159"
       anti_aliasing="$(arg cameras_anti_aliasing)"
+      bounding_boxes="true"
     /> <!-- pixel_format="L8" -->
     <!-- Top-Down camera as moving camera -->

Commit message: bumpers; big room added; cameras at 60 fps; depth at 30

File: urdf/simbot_mecanum_waffle/cameras.urdf.xacro (robot description, xacro)
@@ -2,5 +2,5 @@
 <robot xmlns:xacro="http://ros.org/wiki/xacro" xmlns:gz="http://gazebosim.com/schema">
   <!-- Front / back camera -->
-  <xacro:macro name="robot_camera" params="suffix parent xyz rpy fov:=1.2 width height pixel_format encoder_hw_device encoder_bit_rate encoder_thread_count encoder_input_pixel_format anti_aliasing depth:=false fps:=90 bounding_boxes:=false">
+  <xacro:macro name="robot_camera" params="suffix parent xyz rpy fov:=1.2 width height pixel_format encoder_hw_device encoder_bit_rate encoder_thread_count encoder_input_pixel_format anti_aliasing depth:=false fps:=30 depth_fps:=30 bounding_boxes:=false">
     <link name="camera_link_${suffix}">
       <visual>
@@ -97,5 +97,5 @@
           <pose>0 0 0 0 -${pi/2.0} ${pi/2.0}</pose>
           <always_on>true</always_on>
-          <update_rate>${fps}</update_rate>
+          <update_rate>${depth_fps}</update_rate>
           <visualize>false</visualize>
           <topic>depth_${suffix}/raw</topic>
@@ -109,5 +109,5 @@
             <clip>
               <near>0.1</near> <!-- smaller produces rendering errors -->
-              <far>100</far>
+              <far>10</far>
             </clip>
           </camera>
@@ -117,5 +117,5 @@
   </xacro:macro>
   <!-- top down camera that moves in z direction -->
-  <xacro:macro name="top_down_camera" params="suffix parent xyz rpy width height pixel_format encoder_hw_device encoder_bit_rate encoder_thread_count encoder_input_pixel_format anti_aliasing fps:=90">
+  <xacro:macro name="top_down_camera" params="suffix parent xyz rpy width height pixel_format encoder_hw_device encoder_bit_rate encoder_thread_count encoder_input_pixel_format anti_aliasing fps:=30">
     <link name="camera_link_${suffix}"/>
     <joint name="camera_joint_${suffix}" type="fixed">

File: urdf/simbot_mecanum_waffle/simbot_body.urdf.xacro (robot description, xacro)
@@ -3,4 +3,5 @@
   <!-- <xacro:include filename="$(find simbot_gz)/urdf/simbot_mecanum_waffle/simple_wheel.urdf.xacro"/> -->
   <xacro:include filename="$(find simbot_gz)/urdf/simbot_mecanum_waffle/mecanum_wheel.urdf.xacro"/>
+  <xacro:include filename="$(find simbot_gz)/urdf/simbot_mecanum_waffle/simbot_bumper.urdf.xacro"/>
   <xacro:include filename="$(find simbot_gz)/urdf/simbot_mecanum_waffle/cameras.urdf.xacro"/>
   <xacro:include filename="$(find simbot_gz)/urdf/simbot_mecanum_waffle/lidar.urdf.xacro"/>
@@ -11,6 +12,6 @@
   <xacro:property name="base_collision_box_size" value="0.266 0.266 0.094"/>
   <xacro:property name="wheel_z_offset" value="0.047"/>
-  <xacro:property name="front_wheel_x_offset" value="0.025"/>
-  <xacro:property name="rear_wheel_x_offset" value="-0.12"/>
+  <xacro:property name="front_wheel_x_offset" value="0.015"/>
+  <xacro:property name="rear_wheel_x_offset" value="-0.15"/>
   <xacro:property name="left_wheel_y_offset" value="0.157"/>
   <xacro:property name="right_wheel_y_offset" value="${-left_wheel_y_offset}"/>
@@ -23,5 +24,7 @@
   <xacro:arg name="cameras_width" default="1280"/>
   <xacro:arg name="cameras_height" default="720"/>
-  <xacro:arg name="cameras_anti_aliasing" default="4"/>
+  <xacro:arg name="cameras_anti_aliasing" default="2"/>
+  <xacro:arg name="cameras_fps" default="60"/>
+  <xacro:arg name="depth_cameras_fps" default="30"/>
   <xacro:macro name="base_link" params="parent xyz rpy">
     <link name="base_link">
@@ -51,4 +54,6 @@
       <origin xyz="${xyz}" rpy="${rpy}" />
     </joint>
+    <xacro:bumper suffix="front" xyz=".1 0 0.07" rpy="0 0 0" parent="base_link"/>
+    <xacro:bumper suffix="rear" xyz="-.225 0 0.07" rpy="0 0 ${pi}" parent="base_link"/>
     <!-- Wheels -->
     <!-- Front Left -->
@@ -79,6 +84,8 @@
       xyz="0.07 0.0 0.1030" rpy="0 0 0"
       anti_aliasing="$(arg cameras_anti_aliasing)"
+      bounding_boxes="true"
+      fps="$(arg cameras_fps)"
       depth="true"
-      bounding_boxes="true"
+      depth_fps="$(arg depth_cameras_fps)"
     />
     <xacro:robot_camera parent="base_link" suffix="back"
@@ -93,4 +100,5 @@
       anti_aliasing="$(arg cameras_anti_aliasing)"
       bounding_boxes="true"
+      fps="$(arg cameras_fps)"
     /> <!-- pixel_format="L8" -->
     <!-- Top-Down camera as moving camera -->
@@ -105,11 +113,12 @@
       xyz="0.0 0.0 $(arg camera_top_z)" rpy="${pi} 0 -${pi/2}"
       anti_aliasing="$(arg cameras_anti_aliasing)"
+      fps="$(arg cameras_fps)"
     />
     <xacro:lidar parent="base_link" suffix="1" xyz="0.0000 0.0000 .1510" rpy="0 0 0"/>
     <xacro:imu parent="base_link" suffix="1" xyz="0 0 0" rpy="0 0 0"/>
-    <xacro:range_sensor parent="base_link" suffix="fr" xyz="0.065 -0.10 0.08" rpy="0.0 0.0 -0.187"/>
-    <xacro:range_sensor parent="base_link" suffix="fl" xyz="0.065 0.10 0.08" rpy="0.0 0.0 0.187"/>
-    <xacro:range_sensor parent="base_link" suffix="rr" xyz="-0.19 -0.10 0.08" rpy="0.0 0.0 ${3.1416+0.187}"/>
-    <xacro:range_sensor parent="base_link" suffix="rl" xyz="-0.19 0.10 0.08" rpy="0.0 0.0 ${3.1416-0.187}"/>
+    <xacro:range_sensor parent="base_link" suffix="fr" xyz="0.065 -0.10 0.1" rpy="0.0 0.0 -0.187"/>
+    <xacro:range_sensor parent="base_link" suffix="fl" xyz="0.065 0.10 0.1" rpy="0.0 0.0 0.187"/>
+    <xacro:range_sensor parent="base_link" suffix="rr" xyz="-0.19 -0.10 0.1" rpy="0.0 0.0 ${3.1416+0.187}"/>
+    <xacro:range_sensor parent="base_link" suffix="rl" xyz="-0.19 0.10 0.1" rpy="0.0 0.0 ${3.1416-0.187}"/>
   </xacro:macro>
 </robot>

Commit message: construction cones; camera fps settings

File: urdf/simbot_mecanum_waffle/cameras.urdf.xacro (robot description, xacro)
@@ -2,5 +2,5 @@
 <robot xmlns:xacro="http://ros.org/wiki/xacro" xmlns:gz="http://gazebosim.com/schema">
   <!-- Front / back camera -->
-  <xacro:macro name="robot_camera" params="suffix parent xyz rpy fov:=1.2 width height pixel_format encoder_hw_device encoder_bit_rate encoder_thread_count encoder_input_pixel_format anti_aliasing depth:=false fps:=30 depth_fps:=30 bounding_boxes:=false">
+  <xacro:macro name="robot_camera" params="suffix parent xyz rpy fov:=1.2 width height pixel_format encoder_hw_device encoder_bit_rate encoder_thread_count encoder_input_pixel_format anti_aliasing depth:=false fps:=60 depth_fps:=30 bb_fps:=20 bounding_boxes:=false">
     <link name="camera_link_${suffix}">
       <visual>
@@ -64,5 +64,5 @@
           <always_on>true</always_on>
           <pose>0 0 0 0 -${pi/2.0} ${pi/2.0}</pose>
-          <update_rate>${fps}</update_rate>
+          <update_rate>${bb_fps}</update_rate>
           <visualize>true</visualize>
           <topic>bb_${suffix}/this_must_be_here</topic>
@@ -78,5 +78,5 @@
             <clip>
               <near>0.001</near>
-              <far>10</far>
+              <far>4</far>
             </clip>
           </camera>

File: urdf/simbot_mecanum_waffle/simbot_body.urdf.xacro (robot description, xacro)
@@ -27,4 +27,5 @@
   <xacro:arg name="cameras_fps" default="60"/>
   <xacro:arg name="depth_cameras_fps" default="30"/>
+  <xacro:arg name="bb_cameras_fps" default="30"/>
   <xacro:macro name="base_link" params="parent xyz rpy">
     <link name="base_link">
@@ -88,4 +89,5 @@
       depth="true"
       depth_fps="$(arg depth_cameras_fps)"
+      bb_fps="$(arg bb_cameras_fps)"
     />
     <xacro:robot_camera parent="base_link" suffix="back"

Commit message: fixed mecanum wheels, more models, slope test

File: urdf/simbot_mecanum_waffle/cameras.urdf.xacro (robot description, xacro)
@@ -2,5 +2,5 @@
 <robot xmlns:xacro="http://ros.org/wiki/xacro" xmlns:gz="http://gazebosim.com/schema">
   <!-- Front / back camera -->
-  <xacro:macro name="robot_camera" params="suffix parent xyz rpy fov:=1.2 width height pixel_format encoder_hw_device encoder_bit_rate encoder_thread_count encoder_input_pixel_format anti_aliasing depth:=false fps:=60 depth_fps:=30 bb_fps:=20 bounding_boxes:=false">
+  <xacro:macro name="robot_camera" params="suffix parent xyz rpy fov:=1.2 width height pixel_format encoder_hw_device encoder_bit_rate encoder_thread_count encoder_input_pixel_format anti_aliasing depth:=false depth_width:=640 depth_height:=480 fps:=60 depth_fps:=30 bb_fps:=20 bounding_boxes:=false">
     <link name="camera_link_${suffix}">
       <visual>
@@ -78,5 +78,5 @@
             <clip>
               <near>0.001</near>
-              <far>4</far>
+              <far>7</far>
             </clip>
           </camera>
@@ -104,10 +104,10 @@
             <horizontal_fov>${fov}</horizontal_fov>
             <image>
-              <width>640</width>
-              <height>480</height>
+              <width>${depth_width}</width>
+              <height>${depth_height}</height>
             </image>
             <clip>
               <near>0.1</near> <!-- smaller produces rendering errors -->
-              <far>10</far>
+              <far>100</far>
             </clip>
           </camera>

File: urdf/simbot_mecanum_waffle/mecanum_wheel.urdf.xacro (robot description, xacro)
@@ -16,21 +16,21 @@
     <!-- Assign meshes and friction directions based on suffix -->
     <xacro:if value="${suffix_param == 'fl'}">
-      <xacro:property name="mesh" value="package://simbot_gz/meshes/mecanum_a.dae"/>
+      <xacro:property name="mesh" value="package://simbot_gz/meshes/mecanum_b.dae"/>
       <xacro:property name="visual_rotation" value="0.0"/>
       <xacro:property name="fdir" value="1 -1 0"/>
     </xacro:if>
     <xacro:if value="${suffix_param == 'fr'}">
-      <xacro:property name="mesh" value="package://simbot_gz/meshes/mecanum_b.dae"/>
+      <xacro:property name="mesh" value="package://simbot_gz/meshes/mecanum_a.dae"/>
       <xacro:property name="visual_rotation" value="0.0"/>
       <xacro:property name="fdir" value="1 1 0"/>
     </xacro:if>
     <xacro:if value="${suffix_param == 'rl'}">
-      <xacro:property name="mesh" value="package://simbot_gz/meshes/mecanum_b.dae"/>
-      <xacro:property name="visual_rotation" value="0.0"/>
+      <xacro:property name="mesh" value="package://simbot_gz/meshes/mecanum_a.dae"/>
+      <xacro:property name="visual_rotation" value="${pi}"/>
       <xacro:property name="fdir" value="1 1 0"/>
     </xacro:if>
     <xacro:if value="${suffix_param == 'rr'}">
-      <xacro:property name="mesh" value="package://simbot_gz/meshes/mecanum_a.dae"/>
-      <xacro:property name="visual_rotation" value="0.0"/>
+      <xacro:property name="mesh" value="package://simbot_gz/meshes/mecanum_b.dae"/>
+      <xacro:property name="visual_rotation" value="${pi}"/>
       <xacro:property name="fdir" value="1 -1 0"/>
     </xacro:if>
@@ -47,5 +47,5 @@
     <link name="mecanum_wheel_link_${suffix}">
       <visual>
-        <origin xyz="0.0 0.0 0.0" rpy="0.0 0.0 ${ visual_rotation- pi}"/>
+        <origin xyz="0.0 0.0 0.0" rpy="0.0 0.0 ${visual_rotation-pi}"/>
         <geometry>
           <mesh filename="${mesh}" scale="1.0 1.0 1.0"/>

File: urdf/simbot_mecanum_waffle/simbot_body.urdf.xacro (robot description, xacro)
@@ -27,9 +27,11 @@
   <xacro:arg name="cameras_fps" default="60"/>
   <xacro:arg name="depth_cameras_fps" default="30"/>
+  <xacro:arg name="depth_cameras_width" default="800"/>
+  <xacro:arg name="depth_cameras_height" default="600"/>
   <xacro:arg name="bb_cameras_fps" default="30"/>
   <xacro:macro name="base_link" params="parent xyz rpy">
     <link name="base_link">
       <visual>
-      <origin xyz="${base_visual_offset}" rpy="0 0 0"/>
+        <origin xyz="${base_visual_offset}" rpy="0 0 0"/>
         <geometry>
           <mesh filename="package://simbot_gz/meshes/simbot_base.dae" scale="1 1 1"/>
@@ -66,5 +68,5 @@
                         xyz="${front_wheel_x_offset} ${right_wheel_y_offset} ${wheel_z_offset}"
                         rpy="0 0 0"/>
-    <!-- Rear Left -->
+     <!-- Rear Left -->
     <xacro:mecanum_wheel parent="base_link" suffix="rl"
                         xyz="${rear_wheel_x_offset} ${left_wheel_y_offset} ${wheel_z_offset}"
@@ -88,4 +90,6 @@
       fps="$(arg cameras_fps)"
       depth="true"
+      depth_width="$(arg depth_cameras_width)"
+      depth_height="$(arg depth_cameras_height)"
       depth_fps="$(arg depth_cameras_fps)"
       bb_fps="$(arg bb_cameras_fps)"
@@ -118,5 +122,5 @@
     />
     <xacro:lidar parent="base_link" suffix="1" xyz="0.0000 0.0000 .1510" rpy="0 0 0"/>
-    <xacro:imu parent="base_link" suffix="1" xyz="0 0 0" rpy="0 0 0"/>
+    <xacro:imu parent="base_link" suffix="1" xyz="-.1 0.1 .1" rpy="-${pi} ${pi} -${pi/2}"/>
     <xacro:range_sensor parent="base_link" suffix="fr" xyz="0.065 -0.10 0.1" rpy="0.0 0.0 -0.187"/>
     <xacro:range_sensor parent="base_link" suffix="fl" xyz="0.065 0.10 0.1" rpy="0.0 0.0 0.187"/>
