Commit message: renamed to phntm_gazebo

File: urdf/simbot_mecanum_waffle/cameras.urdf.xacro (robot description, xacro)
@@ -7,5 +7,5 @@
         <origin rpy="0 0 ${pi}"/>
         <geometry>
-          <mesh filename="package://simbot_gz/meshes/camera.dae" />
+          <mesh filename="package://phntm_gazebo/meshes/camera.dae" />
         </geometry>
       </visual>

File: urdf/simbot_mecanum_waffle/gazebo_plugins.urdf.xacro (robot description, xacro)
@@ -7,5 +7,5 @@
     <plugin name="gz::sim::systems::Imu" filename="gz-sim-imu-system" />
     <plugin name="gz_ros2_control::GazeboSimROS2ControlPlugin" filename="gz_ros2_control-system">
-      <parameters>$(find simbot_gz)/config/controller_config_simbot.yaml</parameters>
+      <parameters>$(find phntm_gazebo)/config/controller_config_simbot.yaml</parameters>
     </plugin>
   </gazebo>

File: urdf/simbot_mecanum_waffle/main.urdf.xacro (robot description, xacro)
@@ -1,7 +1,7 @@
 <?xml version="1.0"?>
 <robot name="phntm_simbot" xmlns:xacro="http://ros.org/wiki/xacro" xmlns:gz="http://gazebosim.com/schema">
-  <xacro:include filename="$(find simbot_gz)/urdf/simbot_mecanum_waffle/gazebo_plugins.urdf.xacro" />
-  <xacro:include filename="$(find simbot_gz)/urdf/simbot_mecanum_waffle/simbot_body.urdf.xacro" />
-  <xacro:include filename="$(find simbot_gz)/urdf/simbot_mecanum_waffle/ros2_control.urdf.xacro" />
+  <xacro:include filename="$(find phntm_gazebo)/urdf/simbot_mecanum_waffle/gazebo_plugins.urdf.xacro" />
+  <xacro:include filename="$(find phntm_gazebo)/urdf/simbot_mecanum_waffle/simbot_body.urdf.xacro" />
+  <xacro:include filename="$(find phntm_gazebo)/urdf/simbot_mecanum_waffle/ros2_control.urdf.xacro" />
   <link name="base_footprint" />
   <!-- <link name="base_link" /> -->

File: urdf/simbot_mecanum_waffle/mecanum_wheel.urdf.xacro (robot description, xacro)
@@ -12,24 +12,24 @@
     <xacro:property name="izz" value="0.000111"/>
     <xacro:property name="visual_rotation" value="0.0"/> <!-- might be updated-->
-     <xacro:property name="mesh" value="package://simbot_gz/meshes/3w_v2/omni_frame.stl"/> <!-- might be updated-->
+     <xacro:property name="mesh" value="package://phntm_gazebo/meshes/3w_v2/omni_frame.stl"/> <!-- might be updated-->
      <xacro:property name="fdir" value="1.0 -1.0 0.0"/> <!-- might be updated-->
     <!-- Assign meshes and friction directions based on suffix -->
     <xacro:if value="${suffix_param == 'fl'}">
-      <xacro:property name="mesh" value="package://simbot_gz/meshes/mecanum_b.dae"/>
+      <xacro:property name="mesh" value="package://phntm_gazebo/meshes/mecanum_b.dae"/>
       <xacro:property name="visual_rotation" value="0.0"/>
       <xacro:property name="fdir" value="1 -1 0"/>
     </xacro:if>
     <xacro:if value="${suffix_param == 'fr'}">
-      <xacro:property name="mesh" value="package://simbot_gz/meshes/mecanum_a.dae"/>
+      <xacro:property name="mesh" value="package://phntm_gazebo/meshes/mecanum_a.dae"/>
       <xacro:property name="visual_rotation" value="0.0"/>
       <xacro:property name="fdir" value="1 1 0"/>
     </xacro:if>
     <xacro:if value="${suffix_param == 'rl'}">
-      <xacro:property name="mesh" value="package://simbot_gz/meshes/mecanum_a.dae"/>
+      <xacro:property name="mesh" value="package://phntm_gazebo/meshes/mecanum_a.dae"/>
       <xacro:property name="visual_rotation" value="${pi}"/>
       <xacro:property name="fdir" value="1 1 0"/>
     </xacro:if>
     <xacro:if value="${suffix_param == 'rr'}">
-      <xacro:property name="mesh" value="package://simbot_gz/meshes/mecanum_b.dae"/>
+      <xacro:property name="mesh" value="package://phntm_gazebo/meshes/mecanum_b.dae"/>
       <xacro:property name="visual_rotation" value="${pi}"/>
       <xacro:property name="fdir" value="1 -1 0"/>

File: urdf/simbot_mecanum_waffle/roller.urdf.xacro (robot description, xacro)
@@ -5,5 +5,5 @@
       <visual>
         <geometry>
-          <mesh filename="package://simbot_gz/meshes/4w/roller.stl" />
+          <mesh filename="package://phntm_gazebo/meshes/4w/roller.stl" />
         </geometry>
         <material name="black">
@@ -13,5 +13,5 @@
       <collision>
         <geometry>
-          <mesh filename="package://simbot_gz/meshes/4w/roller.stl" />
+          <mesh filename="package://phntm_gazebo/meshes/4w/roller.stl" />
         </geometry>
       </collision>

File: urdf/simbot_mecanum_waffle/simbot_body.urdf.xacro (robot description, xacro)
@@ -1,11 +1,11 @@
 <?xml version="1.0"?>
 <robot xmlns:xacro="http://ros.org/wiki/xacro" xmlns:gz="http://gazebosim.com/schema">
-  <!-- <xacro:include filename="$(find simbot_gz)/urdf/simbot_mecanum_waffle/simple_wheel.urdf.xacro"/> -->
-  <xacro:include filename="$(find simbot_gz)/urdf/simbot_mecanum_waffle/mecanum_wheel.urdf.xacro"/>
-  <xacro:include filename="$(find simbot_gz)/urdf/simbot_mecanum_waffle/simbot_bumper.urdf.xacro"/>
-  <xacro:include filename="$(find simbot_gz)/urdf/simbot_mecanum_waffle/cameras.urdf.xacro"/>
-  <xacro:include filename="$(find simbot_gz)/urdf/simbot_mecanum_waffle/lidar.urdf.xacro"/>
-  <xacro:include filename="$(find simbot_gz)/urdf/simbot_mecanum_waffle/range_sensor.urdf.xacro"/>
-  <xacro:include filename="$(find simbot_gz)/urdf/simbot_mecanum_waffle/imu.urdf.xacro"/>
+  <!-- <xacro:include filename="$(find phntm_gazebo)/urdf/simbot_mecanum_waffle/simple_wheel.urdf.xacro"/> -->
+  <xacro:include filename="$(find phntm_gazebo)/urdf/simbot_mecanum_waffle/mecanum_wheel.urdf.xacro"/>
+  <xacro:include filename="$(find phntm_gazebo)/urdf/simbot_mecanum_waffle/simbot_bumper.urdf.xacro"/>
+  <xacro:include filename="$(find phntm_gazebo)/urdf/simbot_mecanum_waffle/cameras.urdf.xacro"/>
+  <xacro:include filename="$(find phntm_gazebo)/urdf/simbot_mecanum_waffle/lidar.urdf.xacro"/>
+  <xacro:include filename="$(find phntm_gazebo)/urdf/simbot_mecanum_waffle/range_sensor.urdf.xacro"/>
+  <xacro:include filename="$(find phntm_gazebo)/urdf/simbot_mecanum_waffle/imu.urdf.xacro"/>
   <xacro:property name="base_visual_offset" value="0 0 0.097"/>
   <xacro:property name="base_collision_offset" value="0 0 0.097"/>
@@ -35,5 +35,5 @@
         <origin xyz="${base_visual_offset}" rpy="0 0 0"/>
         <geometry>
-          <mesh filename="package://simbot_gz/meshes/simbot_base.dae" scale="1 1 1"/>
+          <mesh filename="package://phntm_gazebo/meshes/simbot_base.dae" scale="1 1 1"/>
         </geometry>
       </visual>

File: urdf/simbot_mecanum_waffle/simbot_bumper.urdf.xacro (robot description, xacro)
@@ -6,5 +6,5 @@
         <origin xyz="-0.17 0 0.025" rpy="0 0 ${pi/2}"/>
             <geometry>
-            <mesh filename="package://simbot_gz/meshes/simbot_bumper.dae" scale="1 1 1"/>
+            <mesh filename="package://phntm_gazebo/meshes/simbot_bumper.dae" scale="1 1 1"/>
             </geometry>
         </visual>
